Commit message: Placeholder sensor simulation and bridge configuration

File: src/igvc_description/urdf/sensors.urdf.xacro (robot description, xacro)
@@ -1,22 +1,15 @@
 <?xml version="1.0" ?>
 <robot xmlns:xacro="http://www.ros.org/wiki/xacro">
-    <xacro:arg name="camera_name"   default="oak" />
-    <xacro:arg name="camera_model"  default="OAK-D-POE" />
-    <xacro:arg name="base_frame"    default="oak_base" />
-    <xacro:arg name="parent_frame"  default="oak_parent" />
-    <xacro:arg name="cam_pos_x"     default="0.0" />
-    <xacro:arg name="cam_pos_y"     default="0.0" />
-    <xacro:arg name="cam_pos_z"     default="0.0" />
-    <xacro:arg name="cam_roll"      default="0.0" />
-    <xacro:arg name="cam_pitch"     default="0.0" />
-    <xacro:arg name="cam_yaw"       default="0.0" />
-    <xacro:arg name="rs_compat"     default="true" />
-    <xacro:include filename="$(find depthai_descriptions)/urdf/depthai_descr.urdf.xacro" />
-    <joint name="camera_base_joint" type="fixed">
-        <parent link="base_footprint"/>
-        <child link="oak_parent"/>
-        <origin xyz="0 -0.4 0.95" rpy="0 0 ${pi/2}"/>
+    <xacro:include filename="$(find realsense2_description)/urdf/_d435i.urdf.xacro"/>
+    <xacro:sensor_d435i parent="base_link" use_nominal_extrinsics="false">
+        <origin xyz="0.169586 0.00312814 0.06" rpy="0 0 0"/>
+    </xacro:sensor_d435i>
+    <joint name="camera_optical_link" type="fixed">
+        <origin xyz="0 0 0" rpy="${-pi/2} 0 ${-pi/2}"/>
+        <parent link="camera_link"/>
+        <child link="camera_link_optical"/>
     </joint>
-    <gazebo reference="oak_color_frame">
+    <link name="camera_link_optical"></link>
+    <gazebo reference="camera_link">
         <sensor name="oak_depth" type="depth">
             <pose> 0 0 0 0 0 0 </pose>
@@ -24,5 +17,5 @@
             <update_rate>30</update_rate>
             <always_on>1</always_on>
-            <gz_frame_id>oak_color_optical_frame</gz_frame_id>
+            <gz_frame_id>camera_link_optical</gz_frame_id>
             <camera>
                 <horizontal_fov>1.51843645</horizontal_fov>
@@ -40,5 +33,5 @@
         </sensor>
     </gazebo>
-    <gazebo reference="oak_color_frame">
+    <gazebo reference="camera_link">
         <sensor name="oak_color" type="camera">
             <pose> 0 0 0 0 0 0 </pose>
@@ -46,5 +39,5 @@
             <update_rate>30</update_rate>
             <always_on>1</always_on>
-            <gz_frame_id>oak_color_optical_frame</gz_frame_id>
+            <gz_frame_id>camera_link_optical</gz_frame_id>
             <camera>
                 <horizontal_fov>1.51843645</horizontal_fov>

Commit message: Remove duplicate OAK and position existing camera

File: src/igvc_description/urdf/sensors.urdf.xacro (robot description, xacro)
@@ -1,5 +1,5 @@
 <?xml version="1.0" ?>
 <robot xmlns:xacro="http://www.ros.org/wiki/xacro">
-    <xacro:include filename="$(find depthai_descriptions)/urdf/depthai_descr.urdf.xacro"/>
+    <xacro:include filename="$(find depthai_descriptions)/urdf/include/depthai_macro.urdf.xacro"/>
     <xacro:depthai_camera
         camera_name="oak_depth"
@@ -8,14 +8,14 @@
         parent="base_footprint"
         cam_pos_x="0.0"
-        cam_pos_y="0.0"
-        cam_pos_z="0.0"
+        cam_pos_y="-0.4"
+        cam_pos_z="0.8"
         cam_roll="0.0"
         cam_pitch="0.0"
-        cam_yaw="0.0"
+        cam_yaw="${pi/2}"
         rs_compat="true"
     />
     <joint name="camera_base_joint" type="fixed">
         <parent link="base_footprint"/>
-        <child link="oak-d-base-frame"/>
+        <child link="camera_link"/>
         <origin xyz="0 0 0" rpy="${-pi/2} 0 ${-pi/2}"/>
     </joint>

Commit message: Change oak name, add igvc_robot to sensor xacro

File: src/igvc_description/urdf/sensors.urdf.xacro (robot description, xacro)
@@ -1,7 +1,7 @@
 <?xml version="1.0" ?>
-<robot xmlns:xacro="http://www.ros.org/wiki/xacro">
+<robot xmlns:xacro="http://www.ros.org/wiki/xacro" name="igvc_robot">
     <xacro:include filename="$(find depthai_descriptions)/urdf/include/depthai_macro.urdf.xacro"/>
     <xacro:depthai_camera
-        camera_name="oak_depth"
+        camera_name="oak"
         camera_model="OAK-D-POE"
         base_frame="camera_link"
@@ -20,4 +20,5 @@
         <origin xyz="0 0 0" rpy="${-pi/2} 0 ${-pi/2}"/>
     </joint>
+    <link name="camera_link_optical"></link>
     <joint name="camera_optical_joint" type="fixed">
         <parent link="camera_link"/>
@@ -25,5 +26,4 @@
         <origin xyz="0 0 0" rpy="${-pi/2} 0 ${-pi/2}"/>
     </joint>
-    <link name="camera_link_optical"></link>
     <gazebo reference="camera_link">
         <sensor name="oak_depth" type="depth">

Commit message: Reconfigure OAK simulation URDF

File: src/igvc_description/urdf/sensors.urdf.xacro (robot description, xacro)
@@ -4,25 +4,19 @@
     <xacro:arg name="camera_model"  default="OAK-D-POE" />
     <xacro:arg name="base_frame"    default="oak_base" />
-    <xacro:arg name="parent_frame"  default="camera_link" />
+    <xacro:arg name="parent_frame"  default="oak_parent" />
     <xacro:arg name="cam_pos_x"     default="0.0" />
-    <xacro:arg name="cam_pos_y"     default="-0.4" />
-    <xacro:arg name="cam_pos_z"     default="0.8" />
+    <xacro:arg name="cam_pos_y"     default="0.0" />
+    <xacro:arg name="cam_pos_z"     default="0.0" />
     <xacro:arg name="cam_roll"      default="0.0" />
     <xacro:arg name="cam_pitch"     default="0.0" />
-    <xacro:arg name="cam_yaw"       default="${pi/2}" />
+    <xacro:arg name="cam_yaw"       default="0.0" />
     <xacro:arg name="rs_compat"     default="true" />
     <xacro:include filename="$(find depthai_descriptions)/urdf/depthai_descr.urdf.xacro" />
     <joint name="camera_base_joint" type="fixed">
         <parent link="base_footprint"/>
-        <child link="camera_link"/>
-        <origin xyz="0 0 0" rpy="${-pi/2} 0 ${-pi/2}"/>
+        <child link="oak_parent"/>
+        <origin xyz="0 -0.4 0.95" rpy="0 0 ${pi/2}"/>
     </joint>
-    <link name="camera_link_optical"></link>
-    <joint name="camera_optical_joint" type="fixed">
-        <parent link="camera_link"/>
-        <child link="camera_link_optical"/>
-        <origin xyz="0 0 0" rpy="${-pi/2} 0 ${-pi/2}"/>
-    </joint>
-    <gazebo reference="camera_link">
+    <gazebo reference="oak_color_frame">
         <sensor name="oak_depth" type="depth">
             <pose> 0 0 0 0 0 0 </pose>
@@ -30,5 +24,5 @@
             <update_rate>30</update_rate>
             <always_on>1</always_on>
-            <gz_frame_id>camera_link_optical</gz_frame_id>
+            <gz_frame_id>oak_color_optical_frame</gz_frame_id>
             <camera>
                 <horizontal_fov>1.51843645</horizontal_fov>
@@ -46,5 +40,5 @@
         </sensor>
     </gazebo>
-    <gazebo reference="camera_link">
+    <gazebo reference="oak_color_frame">
         <sensor name="oak_color" type="camera">
             <pose> 0 0 0 0 0 0 </pose>
@@ -52,5 +46,5 @@
             <update_rate>30</update_rate>
             <always_on>1</always_on>
-            <gz_frame_id>camera_link_optical</gz_frame_id>
+            <gz_frame_id>oak_color_optical_frame</gz_frame_id>
             <camera>
                 <horizontal_fov>1.51843645</horizontal_fov>

Commit message: Added LIDAR functionality

File: src/igvc_description/urdf/sensors.urdf.xacro (robot description, xacro)
@@ -61,3 +61,47 @@
         </sensor>
     </gazebo>
+    <joint name="laser_joint" type="fixed">
+        <parent link="base_footprint"/>
+        <child link="laser_frame"/>
+        <origin xyz="0 0.2 0.50" rpy="0 0 0"/>
+    </joint>
+    <link name="laser_frame">
+        <visual>
+            <geometry>
+                <cylinder radius="0.0385" length="0.0385"/>
+            </geometry>
+        </visual>
+        <collision>
+            <geometry>
+                <cylinder radius="0.0385" length="0.0385"/>
+            </geometry>
+        </collision>
+        <inertial>
+            <origin xyz="-0.0368571 0.291615 0.214315" rpy="0 0 0"/>
+            <mass value="0.19"/>
+            <inertia ixx="3.60749" ixy="0" ixz="0" iyy="1.28472" iyz="0.159952" izz="3.84124"/>
+        </inertial>
+    </link>
+    <gazebo reference="laser_frame">
+        <sensor name="laser" type="gpu_lidar">
+            <pose> 0 0 0 0 0 0 </pose>
+            <visualize>true</visualize>
+            <update_rate>10</update_rate>
+            <lidar>
+                <scan>
+                    <horizontal>
+                        <samples>360</samples>
+                        <min_angle>-3.14</min_angle>
+                        <max_angle>3.14</max_angle>
+                    </horizontal>
+                </scan>
+                <range>
+                    <min>0.3</min>
+                    <max>12</max>
+                </range>
+            </lidar>
+            <topic>scan</topic>
+            <gz_frame_id>laser_frame</gz_frame_id>
+        </sensor>
+    </gazebo>
 </robot>

Commit message: Reconfigure camera simulation

File: src/igvc_description/urdf/sensors.urdf.xacro (robot description, xacro)
@@ -22,5 +22,5 @@
             <pose> 0 0 0 0 0 0 </pose>
             <topic>oak/depth</topic>
-            <update_rate>30</update_rate>
+            <update_rate>20</update_rate>
             <always_on>1</always_on>
             <gz_frame_id>oak_color_optical_frame</gz_frame_id>
@@ -41,24 +41,40 @@
     </gazebo>
     <gazebo reference="oak_color_frame">
-        <sensor name="oak_color" type="camera">
-            <pose> 0 0 0 0 0 0 </pose>
-            <topic>oak/color</topic>
-            <update_rate>30</update_rate>
-            <always_on>1</always_on>
-            <gz_frame_id>oak_color_optical_frame</gz_frame_id>
+        <sensor name="camera" type="camera">
             <camera>
                 <horizontal_fov>1.51843645</horizontal_fov>
                 <image>
-                    <format>R8G8B8</format>
                     <width>1280</width>
                     <height>720</height>
+                    <format>R8G8B8</format>
                 </image>
                 <clip>
                     <near>0.05</near>
-                    <far>100</far>
+                    <far>20</far>
                 </clip>
+                <noise>
+                    <type>gaussian</type>
+                    <!-- Noise is sampled independently per pixel on each frame.
+                        That pixel's noise value is added to each of its color
+                        channels, which at that point lie in the range [0,1]. -->
+                    <mean>0.0</mean>
+                    <stddev>0.007</stddev>
+                </noise>
+                <optical_frame_id>camera_link_optical</optical_frame_id>
+                <camera_info_topic>camera/camera_info</camera_info_topic>
             </camera>
+            <always_on>1</always_on>
+            <update_rate>20</update_rate>
+            <visualize>true</visualize>
+            <topic>oak/color</topic>
         </sensor>
     </gazebo>
+    <joint name="imu_joint" type="fixed">
+        <origin xyz="0 0 0" rpy="0 0 0" />
+        <parent link="base_link"/>
+        <child link="imu_link" />
+        </joint>
+        <link name="imu_link">
+    </link>
     <joint name="laser_joint" type="fixed">
         <parent link="base_footprint"/>

Commit message: implement sensors, split into separate URDF files

File: src/igvc_description/urdf/sensors.urdf.xacro (robot description, xacro)
@@ -1,123 +1,7 @@
 <?xml version="1.0" ?>
 <robot xmlns:xacro="http://www.ros.org/wiki/xacro">
-    <xacro:arg name="camera_name"   default="oak" />
-    <xacro:arg name="camera_model"  default="OAK-D-POE" />
-    <xacro:arg name="base_frame"    default="oak_base" />
-    <xacro:arg name="parent_frame"  default="oak_parent" />
-    <xacro:arg name="cam_pos_x"     default="0.0" />
-    <xacro:arg name="cam_pos_y"     default="0.0" />
-    <xacro:arg name="cam_pos_z"     default="0.0" />
-    <xacro:arg name="cam_roll"      default="0.0" />
-    <xacro:arg name="cam_pitch"     default="0.0" />
-    <xacro:arg name="cam_yaw"       default="0.0" />
-    <xacro:arg name="rs_compat"     default="true" />
-    <xacro:include filename="$(find depthai_descriptions)/urdf/depthai_descr.urdf.xacro" />
-    <joint name="camera_base_joint" type="fixed">
-        <parent link="base_footprint"/>
-        <child link="oak_parent"/>
-        <origin xyz="0 -0.4 0.95" rpy="0 0 ${pi/2}"/>
-    </joint>
-    <gazebo reference="oak_color_frame">
-        <sensor name="oak_depth" type="depth">
-            <pose> 0 0 0 0 0 0 </pose>
-            <topic>oak/depth</topic>
-            <update_rate>20</update_rate>
-            <always_on>1</always_on>
-            <gz_frame_id>oak_color_optical_frame</gz_frame_id>
-            <camera>
-                <horizontal_fov>1.51843645</horizontal_fov>
-                <image>
-                    <format>R_FLOAT32</format>
-                    <width>1280</width>
-                    <height>720</height>
-                </image>
-                <clip>
-                    <near>0.28</near>
-                    <far>10</far>
-                </clip>
-            </camera>
-            <plugin filename="libgz-sim8-sensors-system.so" name="gz::sim::v8::systems::Sensors"></plugin>
-        </sensor>
-    </gazebo>
-    <gazebo reference="oak_color_frame">
-        <sensor name="camera" type="camera">
-            <camera>
-                <horizontal_fov>1.51843645</horizontal_fov>
-                <image>
-                    <width>1280</width>
-                    <height>720</height>
-                    <format>R8G8B8</format>
-                </image>
-                <clip>
-                    <near>0.05</near>
-                    <far>20</far>
-                </clip>
-                <noise>
-                    <type>gaussian</type>
-                    <!-- Noise is sampled independently per pixel on each frame.
-                        That pixel's noise value is added to each of its color
-                        channels, which at that point lie in the range [0,1]. -->
-                    <mean>0.0</mean>
-                    <stddev>0.007</stddev>
-                </noise>
-                <optical_frame_id>camera_link_optical</optical_frame_id>
-                <camera_info_topic>camera/camera_info</camera_info_topic>
-            </camera>
-            <always_on>1</always_on>
-            <update_rate>20</update_rate>
-            <visualize>true</visualize>
-            <topic>oak/color</topic>
-        </sensor>
-    </gazebo>
-    <joint name="imu_joint" type="fixed">
-        <origin xyz="0 0 0" rpy="0 0 0" />
-        <parent link="base_link"/>
-        <child link="imu_link" />
-        </joint>
-        <link name="imu_link">
-    </link>
-    <joint name="laser_joint" type="fixed">
-        <parent link="base_footprint"/>
-        <child link="laser_frame"/>
-        <origin xyz="0 0.2 0.50" rpy="0 0 0"/>
-    </joint>
-    <link name="laser_frame">
-        <visual>
-            <geometry>
-                <cylinder radius="0.0385" length="0.0385"/>
-            </geometry>
-        </visual>
-        <collision>
-            <geometry>
-                <cylinder radius="0.0385" length="0.0385"/>
-            </geometry>
-        </collision>
-        <inertial>
-            <origin xyz="-0.0368571 0.291615 0.214315" rpy="0 0 0"/>
-            <mass value="0.19"/>
-            <inertia ixx="3.60749" ixy="0" ixz="0" iyy="1.28472" iyz="0.159952" izz="3.84124"/>
-        </inertial>
-    </link>
-    <gazebo reference="laser_frame">
-        <sensor name="laser" type="gpu_lidar">
-            <pose> 0 0 0 0 0 0 </pose>
-            <visualize>true</visualize>
-            <update_rate>10</update_rate>
-            <lidar>
-                <scan>
-                    <horizontal>
-                        <samples>360</samples>
-                        <min_angle>-3.14</min_angle>
-                        <max_angle>3.14</max_angle>
-                    </horizontal>
-                </scan>
-                <range>
-                    <min>0.3</min>
-                    <max>12</max>
-                </range>
-            </lidar>
-            <topic>scan</topic>
-            <gz_frame_id>laser_frame</gz_frame_id>
-        </sensor>
-    </gazebo>
+    <xacro:include filename="$(find igvc_description)/urdf/sensor/lidar.urdf.xacro"/>
+    <xacro:include filename="$(find igvc_description)/urdf/sensor/camera.urdf.xacro"/>
+    <xacro:include filename="$(find igvc_description)/urdf/sensor/imu.urdf.xacro"/>
+    <xacro:include filename="$(find igvc_description)/urdf/sensor/gps.urdf.xacro"/>
 </robot>

Commit message: Added LIDAR functionality (#54)
* Added LIDAR functionality

* Fixed rviz2 crashing issue by adding CycloneDDS

* Adjusted scan range to match Slamtec RPLIDAR S2E

* Fixed cyclonedds implementation.

File: src/igvc_description/urdf/sensors.urdf.xacro (robot description, xacro)
@@ -61,3 +61,47 @@
         </sensor>
     </gazebo>
+    <joint name="laser_joint" type="fixed">
+        <parent link="base_footprint"/>
+        <child link="laser_frame"/>
+        <origin xyz="0 0.2 0.50" rpy="0 0 0"/>
+    </joint>
+    <link name="laser_frame">
+        <visual>
+            <geometry>
+                <cylinder radius="0.0385" length="0.0385"/>
+            </geometry>
+        </visual>
+        <collision>
+            <geometry>
+                <cylinder radius="0.0385" length="0.0385"/>
+            </geometry>
+        </collision>
+        <inertial>
+            <origin xyz="-0.0368571 0.291615 0.214315" rpy="0 0 0"/>
+            <mass value="0.19"/>
+            <inertia ixx="3.60749" ixy="0" ixz="0" iyy="1.28472" iyz="0.159952" izz="3.84124"/>
+        </inertial>
+    </link>
+    <gazebo reference="laser_frame">
+        <sensor name="laser" type="gpu_lidar">
+            <pose> 0 0 0 0 0 0 </pose>
+            <visualize>true</visualize>
+            <update_rate>10</update_rate>
+            <lidar>
+                <scan>
+                    <horizontal>
+                        <samples>360</samples>
+                        <min_angle>-3.14</min_angle>
+                        <max_angle>3.14</max_angle>
+                    </horizontal>
+                </scan>
+                <range>
+                    <min>0.05</min>
+                    <max>30</max>
+                </range>
+            </lidar>
+            <topic>scan</topic>
+            <gz_frame_id>laser_frame</gz_frame_id>
+        </sensor>
+    </gazebo>
 </robot>
