Commit message: Implement remaining parts of sensor suite in simulation (#60)
* Added LIDAR functionality

* Reconfigure camera simulation

* implement sensors, split into separate URDF files

* Fix GPS coordinate definition

* Fixed camera urdf and updated lidar values.

* Updated GPS values to match IGVC location.

---------

Co-authored-by: masshu0504 <mjdavis0504@gmail.com>

File: src/igvc_description/urdf/sensors.urdf.xacro (robot description, xacro)
@@ -1,107 +1,7 @@
 <?xml version="1.0" ?>
 <robot xmlns:xacro="http://www.ros.org/wiki/xacro">
-    <xacro:arg name="camera_name"   default="oak" />
-    <xacro:arg name="camera_model"  default="OAK-D-POE" />
-    <xacro:arg name="base_frame"    default="oak_base" />
-    <xacro:arg name="parent_frame"  default="oak_parent" />
-    <xacro:arg name="cam_pos_x"     default="0.0" />
-    <xacro:arg name="cam_pos_y"     default="0.0" />
-    <xacro:arg name="cam_pos_z"     default="0.0" />
-    <xacro:arg name="cam_roll"      default="0.0" />
-    <xacro:arg name="cam_pitch"     default="0.0" />
-    <xacro:arg name="cam_yaw"       default="0.0" />
-    <xacro:arg name="rs_compat"     default="true" />
-    <xacro:include filename="$(find depthai_descriptions)/urdf/depthai_descr.urdf.xacro" />
-    <joint name="camera_base_joint" type="fixed">
-        <parent link="base_footprint"/>
-        <child link="oak_parent"/>
-        <origin xyz="0 -0.4 0.95" rpy="0 0 ${pi/2}"/>
-    </joint>
-    <gazebo reference="oak_color_frame">
-        <sensor name="oak_depth" type="depth">
-            <pose> 0 0 0 0 0 0 </pose>
-            <topic>oak/depth</topic>
-            <update_rate>30</update_rate>
-            <always_on>1</always_on>
-            <gz_frame_id>oak_color_optical_frame</gz_frame_id>
-            <camera>
-                <horizontal_fov>1.51843645</horizontal_fov>
-                <image>
-                    <format>R_FLOAT32</format>
-                    <width>1280</width>
-                    <height>720</height>
-                </image>
-                <clip>
-                    <near>0.28</near>
-                    <far>10</far>
-                </clip>
-            </camera>
-            <plugin filename="libgz-sim8-sensors-system.so" name="gz::sim::v8::systems::Sensors"></plugin>
-        </sensor>
-    </gazebo>
-    <gazebo reference="oak_color_frame">
-        <sensor name="oak_color" type="camera">
-            <pose> 0 0 0 0 0 0 </pose>
-            <topic>oak/color</topic>
-            <update_rate>30</update_rate>
-            <always_on>1</always_on>
-            <gz_frame_id>oak_color_optical_frame</gz_frame_id>
-            <camera>
-                <horizontal_fov>1.51843645</horizontal_fov>
-                <image>
-                    <format>R8G8B8</format>
-                    <width>1280</width>
-                    <height>720</height>
-                </image>
-                <clip>
-                    <near>0.05</near>
-                    <far>100</far>
-                </clip>
-            </camera>
-        </sensor>
-    </gazebo>
-    <joint name="laser_joint" type="fixed">
-        <parent link="base_footprint"/>
-        <child link="laser_frame"/>
-        <origin xyz="0 0.2 0.50" rpy="0 0 0"/>
-    </joint>
-    <link name="laser_frame">
-        <visual>
-            <geometry>
-                <cylinder radius="0.0385" length="0.0385"/>
-            </geometry>
-        </visual>
-        <collision>
-            <geometry>
-                <cylinder radius="0.0385" length="0.0385"/>
-            </geometry>
-        </collision>
-        <inertial>
-            <origin xyz="-0.0368571 0.291615 0.214315" rpy="0 0 0"/>
-            <mass value="0.19"/>
-            <inertia ixx="3.60749" ixy="0" ixz="0" iyy="1.28472" iyz="0.159952" izz="3.84124"/>
-        </inertial>
-    </link>
-    <gazebo reference="laser_frame">
-        <sensor name="laser" type="gpu_lidar">
-            <pose> 0 0 0 0 0 0 </pose>
-            <visualize>true</visualize>
-            <update_rate>10</update_rate>
-            <lidar>
-                <scan>
-                    <horizontal>
-                        <samples>360</samples>
-                        <min_angle>-3.14</min_angle>
-                        <max_angle>3.14</max_angle>
-                    </horizontal>
-                </scan>
-                <range>
-                    <min>0.05</min>
-                    <max>30</max>
-                </range>
-            </lidar>
-            <topic>scan</topic>
-            <gz_frame_id>laser_frame</gz_frame_id>
-        </sensor>
-    </gazebo>
+    <xacro:include filename="$(find igvc_description)/urdf/sensor/lidar.urdf.xacro"/>
+    <xacro:include filename="$(find igvc_description)/urdf/sensor/camera.urdf.xacro"/>
+    <xacro:include filename="$(find igvc_description)/urdf/sensor/imu.urdf.xacro"/>
+    <xacro:include filename="$(find igvc_description)/urdf/sensor/gps.urdf.xacro"/>
 </robot>

Commit message: Raise LIDAR position, change refresh

File: src/igvc_description/urdf/sensors.urdf.xacro (robot description, xacro)
@@ -64,5 +64,5 @@
         <parent link="base_footprint"/>
         <child link="laser_frame"/>
-        <origin xyz="0 0.2 0.50" rpy="0 0 0"/>
+        <origin xyz="0 0.2 0.75" rpy="0 0 0"/>
     </joint>
     <link name="laser_frame">
@@ -91,5 +91,5 @@
                 <scan>
                     <horizontal>
-                        <samples>360</samples>
+                        <samples>3200</samples>
                         <min_angle>-3.14</min_angle>
                         <max_angle>3.14</max_angle>

Commit message: Amend sensors.urdf.xacro issue

File: src/igvc_description/urdf/sensors.urdf.xacro (robot description, xacro)
@@ -1,107 +1,7 @@
 <?xml version="1.0" ?>
 <robot xmlns:xacro="http://www.ros.org/wiki/xacro">
-    <xacro:arg name="camera_name"   default="oak" />
-    <xacro:arg name="camera_model"  default="OAK-D-POE" />
-    <xacro:arg name="base_frame"    default="oak_base" />
-    <xacro:arg name="parent_frame"  default="oak_parent" />
-    <xacro:arg name="cam_pos_x"     default="0.0" />
-    <xacro:arg name="cam_pos_y"     default="0.0" />
-    <xacro:arg name="cam_pos_z"     default="0.0" />
-    <xacro:arg name="cam_roll"      default="0.0" />
-    <xacro:arg name="cam_pitch"     default="0.0" />
-    <xacro:arg name="cam_yaw"       default="0.0" />
-    <xacro:arg name="rs_compat"     default="true" />
-    <xacro:include filename="$(find depthai_descriptions)/urdf/depthai_descr.urdf.xacro" />
-    <joint name="camera_base_joint" type="fixed">
-        <parent link="base_footprint"/>
-        <child link="oak_parent"/>
-        <origin xyz="0 -0.4 0.95" rpy="0 0 ${pi/2}"/>
-    </joint>
-    <gazebo reference="oak_color_frame">
-        <sensor name="oak_depth" type="depth">
-            <pose> 0 0 0 0 0 0 </pose>
-            <topic>oak/depth</topic>
-            <update_rate>30</update_rate>
-            <always_on>1</always_on>
-            <gz_frame_id>oak_color_optical_frame</gz_frame_id>
-            <camera>
-                <horizontal_fov>1.51843645</horizontal_fov>
-                <image>
-                    <format>R_FLOAT32</format>
-                    <width>1280</width>
-                    <height>720</height>
-                </image>
-                <clip>
-                    <near>0.28</near>
-                    <far>10</far>
-                </clip>
-            </camera>
-            <plugin filename="libgz-sim8-sensors-system.so" name="gz::sim::v8::systems::Sensors"></plugin>
-        </sensor>
-    </gazebo>
-    <gazebo reference="oak_color_frame">
-        <sensor name="oak_color" type="camera">
-            <pose> 0 0 0 0 0 0 </pose>
-            <topic>oak/color</topic>
-            <update_rate>30</update_rate>
-            <always_on>1</always_on>
-            <gz_frame_id>oak_color_optical_frame</gz_frame_id>
-            <camera>
-                <horizontal_fov>1.51843645</horizontal_fov>
-                <image>
-                    <format>R8G8B8</format>
-                    <width>1280</width>
-                    <height>720</height>
-                </image>
-                <clip>
-                    <near>0.05</near>
-                    <far>100</far>
-                </clip>
-            </camera>
-        </sensor>
-    </gazebo>
-    <joint name="laser_joint" type="fixed">
-        <parent link="base_footprint"/>
-        <child link="laser_frame"/>
-        <origin xyz="0 0.2 0.75" rpy="0 0 0"/>
-    </joint>
-    <link name="laser_frame">
-        <visual>
-            <geometry>
-                <cylinder radius="0.0385" length="0.0385"/>
-            </geometry>
-        </visual>
-        <collision>
-            <geometry>
-                <cylinder radius="0.0385" length="0.0385"/>
-            </geometry>
-        </collision>
-        <inertial>
-            <origin xyz="-0.0368571 0.291615 0.214315" rpy="0 0 0"/>
-            <mass value="0.19"/>
-            <inertia ixx="3.60749" ixy="0" ixz="0" iyy="1.28472" iyz="0.159952" izz="3.84124"/>
-        </inertial>
-    </link>
-    <gazebo reference="laser_frame">
-        <sensor name="laser" type="gpu_lidar">
-            <pose> 0 0 0 0 0 0 </pose>
-            <visualize>true</visualize>
-            <update_rate>10</update_rate>
-            <lidar>
-                <scan>
-                    <horizontal>
-                        <samples>3200</samples>
-                        <min_angle>-3.14</min_angle>
-                        <max_angle>3.14</max_angle>
-                    </horizontal>
-                </scan>
-                <range>
-                    <min>0.05</min>
-                    <max>30</max>
-                </range>
-            </lidar>
-            <topic>scan</topic>
-            <gz_frame_id>laser_frame</gz_frame_id>
-        </sensor>
-    </gazebo>
+    <xacro:include filename="$(find igvc_description)/urdf/sensor/lidar.urdf.xacro"/>
+    <xacro:include filename="$(find igvc_description)/urdf/sensor/camera.urdf.xacro"/>
+    <xacro:include filename="$(find igvc_description)/urdf/sensor/imu.urdf.xacro"/>
+    <xacro:include filename="$(find igvc_description)/urdf/sensor/gps.urdf.xacro"/>
 </robot>
