Commit message: Rename otr urdf to model

File: src/igvc_description/urdf/model.urdf.xacro (robot description, xacro)
@@ -7,6 +7,6 @@
     <inertial>
       <origin xyz="0 0 0" rpy="0 0 0"/>
-      <mass value="1e-03"/>
-      <inertia ixx="1e-03" ixy="0" ixz="0" iyy="1e-03" iyz="0" izz="1e-03"/>
+      <mass value="1e-09"/>
+      <inertia ixx="1e-09" ixy="0" ixz="0" iyy="1e-09" iyz="0" izz="1e-09"/>
     </inertial>
     <!-- Part part_5 -->
@@ -14,5 +14,5 @@
       <origin xyz="0 -0.4572 -0.00635" rpy="0 -0 0"/>
       <geometry>
-        <mesh filename="file://$(find igvc_description)/assets/part_5.stl"/>
+        <mesh filename="package://assets/part_5.stl"/>
       </geometry>
       <material name="part_5_material">
@@ -23,5 +23,5 @@
       <origin xyz="0 -0.4572 -0.00635" rpy="0 -0 0"/>
       <geometry>
-        <mesh filename="file://$(find igvc_description)/assets/part_5.stl"/>
+        <mesh filename="package://assets/part_5.stl"/>
       </geometry>
     </collision>
@@ -30,5 +30,5 @@
       <origin xyz="0 -0.4572 -0.00635" rpy="0 -0 0"/>
       <geometry>
-        <mesh filename="file://$(find igvc_description)/assets/part_4.stl"/>
+        <mesh filename="package://assets/part_4.stl"/>
       </geometry>
       <material name="part_4_material">
@@ -39,5 +39,5 @@
       <origin xyz="0 -0.4572 -0.00635" rpy="0 -0 0"/>
       <geometry>
-        <mesh filename="file://$(find igvc_description)/assets/part_4.stl"/>
+        <mesh filename="package://assets/part_4.stl"/>
       </geometry>
     </collision>
@@ -46,5 +46,5 @@
       <origin xyz="0 -0.4572 -0.00635" rpy="0 -0 0"/>
       <geometry>
-        <mesh filename="file://$(find igvc_description)/assets/part_8.stl"/>
+        <mesh filename="package://assets/part_8.stl"/>
       </geometry>
       <material name="part_8_material">
@@ -55,5 +55,5 @@
       <origin xyz="0 -0.4572 -0.00635" rpy="0 -0 0"/>
       <geometry>
-        <mesh filename="file://$(find igvc_description)/assets/part_8.stl"/>
+        <mesh filename="package://assets/part_8.stl"/>
       </geometry>
     </collision>
@@ -62,5 +62,5 @@
       <origin xyz="0 -0.4572 -0.00635" rpy="0 -0 0"/>
       <geometry>
-        <mesh filename="file://$(find igvc_description)/assets/part_2.stl"/>
+        <mesh filename="package://assets/part_2.stl"/>
       </geometry>
       <material name="part_2_material">
@@ -71,5 +71,5 @@
       <origin xyz="0 -0.4572 -0.00635" rpy="0 -0 0"/>
       <geometry>
-        <mesh filename="file://$(find igvc_description)/assets/part_2.stl"/>
+        <mesh filename="package://assets/part_2.stl"/>
       </geometry>
     </collision>
@@ -78,5 +78,5 @@
       <origin xyz="0 -0.4572 -0.00635" rpy="0 -0 0"/>
       <geometry>
-        <mesh filename="file://$(find igvc_description)/assets/part_6.stl"/>
+        <mesh filename="package://assets/part_6.stl"/>
       </geometry>
       <material name="part_6_material">
@@ -87,5 +87,5 @@
       <origin xyz="0 -0.4572 -0.00635" rpy="0 -0 0"/>
       <geometry>
-        <mesh filename="file://$(find igvc_description)/assets/part_6.stl"/>
+        <mesh filename="package://assets/part_6.stl"/>
       </geometry>
     </collision>
@@ -94,5 +94,5 @@
       <origin xyz="0 -0.4572 -0.00635" rpy="0 -0 0"/>
       <geometry>
-        <mesh filename="file://$(find igvc_description)/assets/part_3.stl"/>
+        <mesh filename="package://assets/part_3.stl"/>
       </geometry>
       <material name="part_3_material">
@@ -103,5 +103,5 @@
       <origin xyz="0 -0.4572 -0.00635" rpy="0 -0 0"/>
       <geometry>
-        <mesh filename="file://$(find igvc_description)/assets/part_3.stl"/>
+        <mesh filename="package://assets/part_3.stl"/>
       </geometry>
     </collision>
@@ -110,5 +110,5 @@
       <origin xyz="0 -0.4572 -0.00635" rpy="0 -0 0"/>
       <geometry>
-        <mesh filename="file://$(find igvc_description)/assets/part_7.stl"/>
+        <mesh filename="package://assets/part_7.stl"/>
       </geometry>
       <material name="part_7_material">
@@ -119,5 +119,5 @@
       <origin xyz="0 -0.4572 -0.00635" rpy="0 -0 0"/>
       <geometry>
-        <mesh filename="file://$(find igvc_description)/assets/part_7.stl"/>
+        <mesh filename="package://assets/part_7.stl"/>
       </geometry>
     </collision>
@@ -126,5 +126,5 @@
       <origin xyz="0 -0.4572 -0.00635" rpy="0 -0 0"/>
       <geometry>
-        <mesh filename="file://$(find igvc_description)/assets/part_1.stl"/>
+        <mesh filename="package://assets/part_1.stl"/>
       </geometry>
       <material name="part_1_material">
@@ -135,5 +135,5 @@
       <origin xyz="0 -0.4572 -0.00635" rpy="0 -0 0"/>
       <geometry>
-        <mesh filename="file://$(find igvc_description)/assets/part_1.stl"/>
+        <mesh filename="package://assets/part_1.stl"/>
       </geometry>
     </collision>
@@ -143,6 +143,6 @@
     <inertial>
       <origin xyz="0 0 0" rpy="0 0 0"/>
-      <mass value="1e-03"/>
-      <inertia ixx="1e-03" ixy="0" ixz="0" iyy="1e-03" iyz="0" izz="1e-03"/>
+      <mass value="1e-09"/>
+      <inertia ixx="1e-09" ixy="0" ixz="0" iyy="1e-09" iyz="0" izz="1e-09"/>
     </inertial>
     <!-- Part part_10 -->
@@ -150,5 +150,5 @@
       <origin xyz="-0.4572 -0 0.2159" rpy="-1.5708 -1.5708 0"/>
       <geometry>
-        <mesh filename="file://$(find igvc_description)/assets/part_10.stl"/>
+        <mesh filename="package://assets/part_10.stl"/>
       </geometry>
       <material name="part_10_material">
@@ -159,5 +159,5 @@
       <origin xyz="-0.4572 -0 0.2159" rpy="-1.5708 -1.5708 0"/>
       <geometry>
-        <mesh filename="file://$(find igvc_description)/assets/part_10.stl"/>
+        <mesh filename="package://assets/part_10.stl"/>
       </geometry>
     </collision>
@@ -175,6 +175,6 @@
     <inertial>
       <origin xyz="0 0 0" rpy="0 0 0"/>
-      <mass value="1e-03"/>
-      <inertia ixx="1e-03" ixy="0" ixz="0" iyy="1e-03" iyz="0" izz="1e-03"/>
+      <mass value="1e-09"/>
+      <inertia ixx="1e-09" ixy="0" ixz="0" iyy="1e-09" iyz="0" izz="1e-09"/>
     </inertial>
     <!-- Part part_9 -->
@@ -182,5 +182,5 @@
       <origin xyz="-0.4572 0 0.2159" rpy="1.5708 1.5708 0"/>
       <geometry>
-        <mesh filename="file://$(find igvc_description)/assets/part_9.stl"/>
+        <mesh filename="package://assets/part_9.stl"/>
       </geometry>
       <material name="part_9_material">
@@ -191,5 +191,5 @@
       <origin xyz="-0.4572 0 0.2159" rpy="1.5708 1.5708 0"/>
       <geometry>
-        <mesh filename="file://$(find igvc_description)/assets/part_9.stl"/>
+        <mesh filename="package://assets/part_9.stl"/>
       </geometry>
     </collision>

Commit message: add package name to URDF meshes (automate this in the future)

File: src/igvc_description/urdf/model.urdf.xacro (robot description, xacro)
@@ -14,5 +14,5 @@
       <origin xyz="0 -0.4572 -0.00635" rpy="0 -0 0"/>
       <geometry>
-        <mesh filename="package://assets/part_5.stl"/>
+        <mesh filename="package://igvc_description/assets/part_5.stl"/>
       </geometry>
       <material name="part_5_material">
@@ -23,5 +23,5 @@
       <origin xyz="0 -0.4572 -0.00635" rpy="0 -0 0"/>
       <geometry>
-        <mesh filename="package://assets/part_5.stl"/>
+        <mesh filename="package://igvc_description/assets/part_5.stl"/>
       </geometry>
     </collision>
@@ -30,5 +30,5 @@
       <origin xyz="0 -0.4572 -0.00635" rpy="0 -0 0"/>
       <geometry>
-        <mesh filename="package://assets/part_4.stl"/>
+        <mesh filename="package://igvc_description/assets/part_4.stl"/>
       </geometry>
       <material name="part_4_material">
@@ -39,5 +39,5 @@
       <origin xyz="0 -0.4572 -0.00635" rpy="0 -0 0"/>
       <geometry>
-        <mesh filename="package://assets/part_4.stl"/>
+        <mesh filename="package://igvc_description/assets/part_4.stl"/>
       </geometry>
     </collision>
@@ -46,5 +46,5 @@
       <origin xyz="0 -0.4572 -0.00635" rpy="0 -0 0"/>
       <geometry>
-        <mesh filename="package://assets/part_8.stl"/>
+        <mesh filename="package://igvc_description/assets/part_8.stl"/>
       </geometry>
       <material name="part_8_material">
@@ -55,5 +55,5 @@
       <origin xyz="0 -0.4572 -0.00635" rpy="0 -0 0"/>
       <geometry>
-        <mesh filename="package://assets/part_8.stl"/>
+        <mesh filename="package://igvc_description/assets/part_8.stl"/>
       </geometry>
     </collision>
@@ -62,5 +62,5 @@
       <origin xyz="0 -0.4572 -0.00635" rpy="0 -0 0"/>
       <geometry>
-        <mesh filename="package://assets/part_2.stl"/>
+        <mesh filename="package://igvc_description/assets/part_2.stl"/>
       </geometry>
       <material name="part_2_material">
@@ -71,5 +71,5 @@
       <origin xyz="0 -0.4572 -0.00635" rpy="0 -0 0"/>
       <geometry>
-        <mesh filename="package://assets/part_2.stl"/>
+        <mesh filename="package://igvc_description/assets/part_2.stl"/>
       </geometry>
     </collision>
@@ -78,5 +78,5 @@
       <origin xyz="0 -0.4572 -0.00635" rpy="0 -0 0"/>
       <geometry>
-        <mesh filename="package://assets/part_6.stl"/>
+        <mesh filename="package://igvc_description/assets/part_6.stl"/>
       </geometry>
       <material name="part_6_material">
@@ -87,5 +87,5 @@
       <origin xyz="0 -0.4572 -0.00635" rpy="0 -0 0"/>
       <geometry>
-        <mesh filename="package://assets/part_6.stl"/>
+        <mesh filename="package://igvc_description/assets/part_6.stl"/>
       </geometry>
     </collision>
@@ -94,5 +94,5 @@
       <origin xyz="0 -0.4572 -0.00635" rpy="0 -0 0"/>
       <geometry>
-        <mesh filename="package://assets/part_3.stl"/>
+        <mesh filename="package://igvc_description/assets/part_3.stl"/>
       </geometry>
       <material name="part_3_material">
@@ -103,5 +103,5 @@
       <origin xyz="0 -0.4572 -0.00635" rpy="0 -0 0"/>
       <geometry>
-        <mesh filename="package://assets/part_3.stl"/>
+        <mesh filename="package://igvc_description/assets/part_3.stl"/>
       </geometry>
     </collision>
@@ -110,5 +110,5 @@
       <origin xyz="0 -0.4572 -0.00635" rpy="0 -0 0"/>
       <geometry>
-        <mesh filename="package://assets/part_7.stl"/>
+        <mesh filename="package://igvc_description/assets/part_7.stl"/>
       </geometry>
       <material name="part_7_material">
@@ -119,5 +119,5 @@
       <origin xyz="0 -0.4572 -0.00635" rpy="0 -0 0"/>
       <geometry>
-        <mesh filename="package://assets/part_7.stl"/>
+        <mesh filename="package://igvc_description/assets/part_7.stl"/>
       </geometry>
     </collision>
@@ -126,5 +126,5 @@
       <origin xyz="0 -0.4572 -0.00635" rpy="0 -0 0"/>
       <geometry>
-        <mesh filename="package://assets/part_1.stl"/>
+        <mesh filename="package://igvc_description/assets/part_1.stl"/>
       </geometry>
       <material name="part_1_material">
@@ -135,5 +135,5 @@
       <origin xyz="0 -0.4572 -0.00635" rpy="0 -0 0"/>
       <geometry>
-        <mesh filename="package://assets/part_1.stl"/>
+        <mesh filename="package://igvc_description/assets/part_1.stl"/>
       </geometry>
     </collision>
@@ -150,5 +150,5 @@
       <origin xyz="-0.4572 -0 0.2159" rpy="-1.5708 -1.5708 0"/>
       <geometry>
-        <mesh filename="package://assets/part_10.stl"/>
+        <mesh filename="package://igvc_description/assets/part_10.stl"/>
       </geometry>
       <material name="part_10_material">
@@ -159,5 +159,5 @@
       <origin xyz="-0.4572 -0 0.2159" rpy="-1.5708 -1.5708 0"/>
       <geometry>
-        <mesh filename="package://assets/part_10.stl"/>
+        <mesh filename="package://igvc_description/assets/part_10.stl"/>
       </geometry>
     </collision>
@@ -182,5 +182,5 @@
       <origin xyz="-0.4572 0 0.2159" rpy="1.5708 1.5708 0"/>
       <geometry>
-        <mesh filename="package://assets/part_9.stl"/>
+        <mesh filename="package://igvc_description/assets/part_9.stl"/>
       </geometry>
       <material name="part_9_material">
@@ -191,5 +191,5 @@
       <origin xyz="-0.4572 0 0.2159" rpy="1.5708 1.5708 0"/>
       <geometry>
-        <mesh filename="package://assets/part_9.stl"/>
+        <mesh filename="package://igvc_description/assets/part_9.stl"/>
       </geometry>
     </collision>

Commit message: Fix file URDF locations

File: src/igvc_description/urdf/model.urdf.xacro (robot description, xacro)
@@ -14,5 +14,5 @@
       <origin xyz="0 -0.4572 -0.00635" rpy="0 -0 0"/>
       <geometry>
-        <mesh filename="package://igvc_description/assets/part_5.stl"/>
+        <mesh filename="file://$(find igvc_description)/assets/part_5.stl"/>
       </geometry>
       <material name="part_5_material">
@@ -23,5 +23,5 @@
       <origin xyz="0 -0.4572 -0.00635" rpy="0 -0 0"/>
       <geometry>
-        <mesh filename="package://igvc_description/assets/part_5.stl"/>
+        <mesh filename="file://$(find igvc_description)/assets/part_5.stl"/>
       </geometry>
     </collision>
@@ -30,5 +30,5 @@
       <origin xyz="0 -0.4572 -0.00635" rpy="0 -0 0"/>
       <geometry>
-        <mesh filename="package://igvc_description/assets/part_4.stl"/>
+        <mesh filename="file://$(find igvc_description)/assets/part_4.stl"/>
       </geometry>
       <material name="part_4_material">
@@ -39,5 +39,5 @@
       <origin xyz="0 -0.4572 -0.00635" rpy="0 -0 0"/>
       <geometry>
-        <mesh filename="package://igvc_description/assets/part_4.stl"/>
+        <mesh filename="file://$(find igvc_description)/assets/part_4.stl"/>
       </geometry>
     </collision>
@@ -46,5 +46,5 @@
       <origin xyz="0 -0.4572 -0.00635" rpy="0 -0 0"/>
       <geometry>
-        <mesh filename="package://igvc_description/assets/part_8.stl"/>
+        <mesh filename="file://$(find igvc_description)/assets/part_8.stl"/>
       </geometry>
       <material name="part_8_material">
@@ -55,5 +55,5 @@
       <origin xyz="0 -0.4572 -0.00635" rpy="0 -0 0"/>
       <geometry>
-        <mesh filename="package://igvc_description/assets/part_8.stl"/>
+        <mesh filename="file://$(find igvc_description)/assets/part_8.stl"/>
       </geometry>
     </collision>
@@ -62,5 +62,5 @@
       <origin xyz="0 -0.4572 -0.00635" rpy="0 -0 0"/>
       <geometry>
-        <mesh filename="package://igvc_description/assets/part_2.stl"/>
+        <mesh filename="file://$(find igvc_description)/assets/part_2.stl"/>
       </geometry>
       <material name="part_2_material">
@@ -71,5 +71,5 @@
       <origin xyz="0 -0.4572 -0.00635" rpy="0 -0 0"/>
       <geometry>
-        <mesh filename="package://igvc_description/assets/part_2.stl"/>
+        <mesh filename="file://$(find igvc_description)/assets/part_2.stl"/>
       </geometry>
     </collision>
@@ -78,5 +78,5 @@
       <origin xyz="0 -0.4572 -0.00635" rpy="0 -0 0"/>
       <geometry>
-        <mesh filename="package://igvc_description/assets/part_6.stl"/>
+        <mesh filename="file://$(find igvc_description)/assets/part_6.stl"/>
       </geometry>
       <material name="part_6_material">
@@ -87,5 +87,5 @@
       <origin xyz="0 -0.4572 -0.00635" rpy="0 -0 0"/>
       <geometry>
-        <mesh filename="package://igvc_description/assets/part_6.stl"/>
+        <mesh filename="file://$(find igvc_description)/assets/part_6.stl"/>
       </geometry>
     </collision>
@@ -94,5 +94,5 @@
       <origin xyz="0 -0.4572 -0.00635" rpy="0 -0 0"/>
       <geometry>
-        <mesh filename="package://igvc_description/assets/part_3.stl"/>
+        <mesh filename="file://$(find igvc_description)/assets/part_3.stl"/>
       </geometry>
       <material name="part_3_material">
@@ -103,5 +103,5 @@
       <origin xyz="0 -0.4572 -0.00635" rpy="0 -0 0"/>
       <geometry>
-        <mesh filename="package://igvc_description/assets/part_3.stl"/>
+        <mesh filename="file://$(find igvc_description)/assets/part_3.stl"/>
       </geometry>
     </collision>
@@ -110,5 +110,5 @@
       <origin xyz="0 -0.4572 -0.00635" rpy="0 -0 0"/>
       <geometry>
-        <mesh filename="package://igvc_description/assets/part_7.stl"/>
+        <mesh filename="file://$(find igvc_description)/assets/part_7.stl"/>
       </geometry>
       <material name="part_7_material">
@@ -119,5 +119,5 @@
       <origin xyz="0 -0.4572 -0.00635" rpy="0 -0 0"/>
       <geometry>
-        <mesh filename="package://igvc_description/assets/part_7.stl"/>
+        <mesh filename="file://$(find igvc_description)/assets/part_7.stl"/>
       </geometry>
     </collision>
@@ -126,5 +126,5 @@
       <origin xyz="0 -0.4572 -0.00635" rpy="0 -0 0"/>
       <geometry>
-        <mesh filename="package://igvc_description/assets/part_1.stl"/>
+        <mesh filename="file://$(find igvc_description)/assets/part_1.stl"/>
       </geometry>
       <material name="part_1_material">
@@ -135,5 +135,5 @@
       <origin xyz="0 -0.4572 -0.00635" rpy="0 -0 0"/>
       <geometry>
-        <mesh filename="package://igvc_description/assets/part_1.stl"/>
+        <mesh filename="file://$(find igvc_description)/assets/part_1.stl"/>
       </geometry>
     </collision>
@@ -150,5 +150,5 @@
       <origin xyz="-0.4572 -0 0.2159" rpy="-1.5708 -1.5708 0"/>
       <geometry>
-        <mesh filename="package://igvc_description/assets/part_10.stl"/>
+        <mesh filename="file://$(find igvc_description)/assets/part_10.stl"/>
       </geometry>
       <material name="part_10_material">
@@ -159,5 +159,5 @@
       <origin xyz="-0.4572 -0 0.2159" rpy="-1.5708 -1.5708 0"/>
       <geometry>
-        <mesh filename="package://igvc_description/assets/part_10.stl"/>
+        <mesh filename="file://$(find igvc_description)/assets/part_10.stl"/>
       </geometry>
     </collision>
@@ -182,5 +182,5 @@
       <origin xyz="-0.4572 0 0.2159" rpy="1.5708 1.5708 0"/>
       <geometry>
-        <mesh filename="package://igvc_description/assets/part_9.stl"/>
+        <mesh filename="file://$(find igvc_description)/assets/part_9.stl"/>
       </geometry>
       <material name="part_9_material">
@@ -191,5 +191,5 @@
       <origin xyz="-0.4572 0 0.2159" rpy="1.5708 1.5708 0"/>
       <geometry>
-        <mesh filename="package://igvc_description/assets/part_9.stl"/>
+        <mesh filename="file://$(find igvc_description)/assets/part_9.stl"/>
       </geometry>
     </collision>

Commit message: Alter inertial values

File: src/igvc_description/urdf/model.urdf.xacro (robot description, xacro)
@@ -7,6 +7,6 @@
     <inertial>
       <origin xyz="0 0 0" rpy="0 0 0"/>
-      <mass value="1e-09"/>
-      <inertia ixx="1e-09" ixy="0" ixz="0" iyy="1e-09" iyz="0" izz="1e-09"/>
+      <mass value="1e-03"/>
+      <inertia ixx="1e-03" ixy="0" ixz="0" iyy="1e-03" iyz="0" izz="1e-03"/>
     </inertial>
     <!-- Part part_5 -->
@@ -143,6 +143,6 @@
     <inertial>
       <origin xyz="0 0 0" rpy="0 0 0"/>
-      <mass value="1e-09"/>
-      <inertia ixx="1e-09" ixy="0" ixz="0" iyy="1e-09" iyz="0" izz="1e-09"/>
+      <mass value="1e-03"/>
+      <inertia ixx="1e-03" ixy="0" ixz="0" iyy="1e-03" iyz="0" izz="1e-03"/>
     </inertial>
     <!-- Part part_10 -->
@@ -175,6 +175,6 @@
     <inertial>
       <origin xyz="0 0 0" rpy="0 0 0"/>
-      <mass value="1e-09"/>
-      <inertia ixx="1e-09" ixy="0" ixz="0" iyy="1e-09" iyz="0" izz="1e-09"/>
+      <mass value="1e-03"/>
+      <inertia ixx="1e-03" ixy="0" ixz="0" iyy="1e-03" iyz="0" izz="1e-03"/>
     </inertial>
     <!-- Part part_9 -->
