Commit message: Update URDF to Low Fidelity V1

File: src/igvc_description/urdf/model.urdf.xacro (robot description, xacro)
@@ -1,5 +1,5 @@
 <?xml version="1.0" ?>
 <!-- Generated using onshape-to-robot -->
-<!-- Onshape https://cad.onshape.com/documents/bd8c1cbb3cbd66454183450f/w/dfd94c9f83ff0fc6c8761109/e/c765fc0d53504544c054bc0a -->
+<!-- Onshape https://cad.onshape.com/documents/bd8c1cbb3cbd66454183450f/w/dfd94c9f83ff0fc6c8761109/e/b8893f818205c61a56339f3e -->
 <robot xmlns:xacro="http://www.ros.org/wiki/xacro">
   <!-- Link part_1 -->
@@ -10,7 +10,343 @@
       <inertia ixx="1e-03" ixy="0" ixz="0" iyy="1e-03" iyz="0" izz="1e-03"/>
     </inertial>
+    <!-- Part part_22 -->
+    <visual>
+      <origin xyz="-0.193704 -0.552769 0.227447" rpy="0 0 0"/>
+      <geometry>
+        <mesh filename="file://$(find igvc_description)/assets/part_22.stl"/>
+      </geometry>
+      <material name="part_22_material">
+        <color rgba="0.647059 0.647059 0.647059 1"/>
+      </material>
+    </visual>
+    <collision>
+      <origin xyz="-0.193704 -0.552769 0.227447" rpy="0 0 0"/>
+      <geometry>
+        <mesh filename="file://$(find igvc_description)/assets/part_22.stl"/>
+      </geometry>
+    </collision>
+    <!-- Part part_3 -->
+    <visual>
+      <origin xyz="-0.193704 -0.552769 0.227447" rpy="0 0 0"/>
+      <geometry>
+        <mesh filename="file://$(find igvc_description)/assets/part_3.stl"/>
+      </geometry>
+      <material name="part_3_material">
+        <color rgba="0.647059 0.647059 0.647059 1"/>
+      </material>
+    </visual>
+    <collision>
+      <origin xyz="-0.193704 -0.552769 0.227447" rpy="0 0 0"/>
+      <geometry>
+        <mesh filename="file://$(find igvc_description)/assets/part_3.stl"/>
+      </geometry>
+    </collision>
+    <!-- Part part_17 -->
+    <visual>
+      <origin xyz="0.0837819 0.221931 0.441433" rpy="-1.5708 -0 -0"/>
+      <geometry>
+        <mesh filename="file://$(find igvc_description)/assets/part_17.stl"/>
+      </geometry>
+      <material name="part_17_material">
+        <color rgba="0.647059 0.647059 0.647059 1"/>
+      </material>
+    </visual>
+    <collision>
+      <origin xyz="0.0837819 0.221931 0.441433" rpy="-1.5708 -0 -0"/>
+      <geometry>
+        <mesh filename="file://$(find igvc_description)/assets/part_17.stl"/>
+      </geometry>
+    </collision>
+    <!-- Part part_27 -->
+    <visual>
+      <origin xyz="-0.193704 -0.552769 0.227447" rpy="0 0 0"/>
+      <geometry>
+        <mesh filename="file://$(find igvc_description)/assets/part_27.stl"/>
+      </geometry>
+      <material name="part_27_material">
+        <color rgba="0.231373 0.380392 0.705882 1"/>
+      </material>
+    </visual>
+    <collision>
+      <origin xyz="-0.193704 -0.552769 0.227447" rpy="0 0 0"/>
+      <geometry>
+        <mesh filename="file://$(find igvc_description)/assets/part_27.stl"/>
+      </geometry>
+    </collision>
+    <!-- Part part_25 -->
+    <visual>
+      <origin xyz="-0.193704 -0.552769 0.227447" rpy="0 0 0"/>
+      <geometry>
+        <mesh filename="file://$(find igvc_description)/assets/part_25.stl"/>
+      </geometry>
+      <material name="part_25_material">
+        <color rgba="0.647059 0.647059 0.647059 1"/>
+      </material>
+    </visual>
+    <collision>
+      <origin xyz="-0.193704 -0.552769 0.227447" rpy="0 0 0"/>
+      <geometry>
+        <mesh filename="file://$(find igvc_description)/assets/part_25.stl"/>
+      </geometry>
+    </collision>
+    <!-- Part part_14 -->
+    <visual>
+      <origin xyz="-0.193704 -0.552769 0.227447" rpy="0 0 0"/>
+      <geometry>
+        <mesh filename="file://$(find igvc_description)/assets/part_14.stl"/>
+      </geometry>
+      <material name="part_14_material">
+        <color rgba="0.647059 0.647059 0.647059 1"/>
+      </material>
+    </visual>
+    <collision>
+      <origin xyz="-0.193704 -0.552769 0.227447" rpy="0 0 0"/>
+      <geometry>
+        <mesh filename="file://$(find igvc_description)/assets/part_14.stl"/>
+      </geometry>
+    </collision>
+    <!-- Part part_9 -->
+    <visual>
+      <origin xyz="-0.193704 -0.552769 0.227447" rpy="0 0 0"/>
+      <geometry>
+        <mesh filename="file://$(find igvc_description)/assets/part_9.stl"/>
+      </geometry>
+      <material name="part_9_material">
+        <color rgba="0.647059 0.647059 0.647059 1"/>
+      </material>
+    </visual>
+    <collision>
+      <origin xyz="-0.193704 -0.552769 0.227447" rpy="0 0 0"/>
+      <geometry>
+        <mesh filename="file://$(find igvc_description)/assets/part_9.stl"/>
+      </geometry>
+    </collision>
+    <!-- Part part_23 -->
+    <visual>
+      <origin xyz="-0.193704 -0.552769 0.227447" rpy="0 0 0"/>
+      <geometry>
+        <mesh filename="file://$(find igvc_description)/assets/part_23.stl"/>
+      </geometry>
+      <material name="part_23_material">
+        <color rgba="0.647059 0.647059 0.647059 1"/>
+      </material>
+    </visual>
+    <collision>
+      <origin xyz="-0.193704 -0.552769 0.227447" rpy="0 0 0"/>
+      <geometry>
+        <mesh filename="file://$(find igvc_description)/assets/part_23.stl"/>
+      </geometry>
+    </collision>
+    <!-- Part part_10 -->
+    <visual>
+      <origin xyz="-0.193704 -0.552769 0.227447" rpy="0 0 0"/>
+      <geometry>
+        <mesh filename="file://$(find igvc_description)/assets/part_10.stl"/>
+      </geometry>
+      <material name="part_10_material">
+        <color rgba="0.647059 0.647059 0.647059 1"/>
+      </material>
+    </visual>
+    <collision>
+      <origin xyz="-0.193704 -0.552769 0.227447" rpy="0 0 0"/>
+      <geometry>
+        <mesh filename="file://$(find igvc_description)/assets/part_10.stl"/>
+      </geometry>
+    </collision>
+    <!-- Part part_24 -->
+    <visual>
+      <origin xyz="-0.193704 -0.552769 0.227447" rpy="0 0 0"/>
+      <geometry>
+        <mesh filename="file://$(find igvc_description)/assets/part_24.stl"/>
+      </geometry>
+      <material name="part_24_material">
+        <color rgba="0.647059 0.647059 0.647059 1"/>
+      </material>
+    </visual>
+    <collision>
+      <origin xyz="-0.193704 -0.552769 0.227447" rpy="0 0 0"/>
+      <geometry>
+        <mesh filename="file://$(find igvc_description)/assets/part_24.stl"/>
+      </geometry>
+    </collision>
+    <!-- Part part_7 -->
+    <visual>
+      <origin xyz="-0.193704 -0.552769 0.227447" rpy="0 0 0"/>
+      <geometry>
+        <mesh filename="file://$(find igvc_description)/assets/part_7.stl"/>
+      </geometry>
+      <material name="part_7_material">
+        <color rgba="0.647059 0.647059 0.647059 1"/>
+      </material>
+    </visual>
+    <collision>
+      <origin xyz="-0.193704 -0.552769 0.227447" rpy="0 0 0"/>
+      <geometry>
+        <mesh filename="file://$(find igvc_description)/assets/part_7.stl"/>
+      </geometry>
+    </collision>
+    <!-- Part part_26 -->
+    <visual>
+      <origin xyz="-0.193704 -0.552769 0.227447" rpy="0 0 0"/>
+      <geometry>
+        <mesh filename="file://$(find igvc_description)/assets/part_26.stl"/>
+      </geometry>
+      <material name="part_26_material">
+        <color rgba="0.647059 0.647059 0.647059 1"/>
+      </material>
+    </visual>
+    <collision>
+      <origin xyz="-0.193704 -0.552769 0.227447" rpy="0 0 0"/>
+      <geometry>
+        <mesh filename="file://$(find igvc_description)/assets/part_26.stl"/>
+      </geometry>
+    </collision>
+    <!-- Part part_1 -->
+    <visual>
+      <origin xyz="-0.193704 -0.552769 0.227447" rpy="0 0 0"/>
+      <geometry>
+        <mesh filename="file://$(find igvc_description)/assets/part_1.stl"/>
+      </geometry>
+      <material name="part_1_material">
+        <color rgba="0.647059 0.647059 0.647059 1"/>
+      </material>
+    </visual>
+    <collision>
+      <origin xyz="-0.193704 -0.552769 0.227447" rpy="0 0 0"/>
+      <geometry>
+        <mesh filename="file://$(find igvc_description)/assets/part_1.stl"/>
+      </geometry>
+    </collision>
+    <!-- Part part_20 -->
+    <visual>
+      <origin xyz="-0.193704 -0.552769 0.227447" rpy="0 0 0"/>
+      <geometry>
+        <mesh filename="file://$(find igvc_description)/assets/part_20.stl"/>
+      </geometry>
+      <material name="part_20_material">
+        <color rgba="0.647059 0.647059 0.647059 1"/>
+      </material>
+    </visual>
+    <collision>
+      <origin xyz="-0.193704 -0.552769 0.227447" rpy="0 0 0"/>
+      <geometry>
+        <mesh filename="file://$(find igvc_description)/assets/part_20.stl"/>
+      </geometry>
+    </collision>
+    <!-- Part part_8 -->
+    <visual>
+      <origin xyz="-0.193704 -0.552769 0.227447" rpy="0 0 0"/>
+      <geometry>
+        <mesh filename="file://$(find igvc_description)/assets/part_8.stl"/>
+      </geometry>
+      <material name="part_8_material">
+        <color rgba="0.647059 0.647059 0.647059 1"/>
+      </material>
+    </visual>
+    <collision>
+      <origin xyz="-0.193704 -0.552769 0.227447" rpy="0 0 0"/>
+      <geometry>
+        <mesh filename="file://$(find igvc_description)/assets/part_8.stl"/>
+      </geometry>
+    </collision>
+    <!-- Part part_6 -->
+    <visual>
+      <origin xyz="-0.193704 -0.552769 0.227447" rpy="0 0 0"/>
+      <geometry>
+        <mesh filename="file://$(find igvc_description)/assets/part_6.stl"/>
+      </geometry>
+      <material name="part_6_material">
+        <color rgba="0.647059 0.647059 0.647059 1"/>
+      </material>
+    </visual>
+    <collision>
+      <origin xyz="-0.193704 -0.552769 0.227447" rpy="0 0 0"/>
+      <geometry>
+        <mesh filename="file://$(find igvc_description)/assets/part_6.stl"/>
+      </geometry>
+    </collision>
+    <!-- Part part_12 -->
+    <visual>
+      <origin xyz="-0.193704 -0.552769 0.227447" rpy="0 0 0"/>
+      <geometry>
+        <mesh filename="file://$(find igvc_description)/assets/part_12.stl"/>
+      </geometry>
+      <material name="part_12_material">
+        <color rgba="0.647059 0.647059 0.647059 1"/>
+      </material>
+    </visual>
+    <collision>
+      <origin xyz="-0.193704 -0.552769 0.227447" rpy="0 0 0"/>
+      <geometry>
+        <mesh filename="file://$(find igvc_description)/assets/part_12.stl"/>
+      </geometry>
+    </collision>
+    <!-- Part part_21 -->
+    <visual>
+      <origin xyz="-0.193704 -0.552769 0.227447" rpy="0 0 0"/>
+      <geometry>
+        <mesh filename="file://$(find igvc_description)/assets/part_21.stl"/>
+      </geometry>
+      <material name="part_21_material">
+        <color rgba="0.647059 0.647059 0.647059 1"/>
+      </material>
+    </visual>
+    <collision>
+      <origin xyz="-0.193704 -0.552769 0.227447" rpy="0 0 0"/>
+      <geometry>
+        <mesh filename="file://$(find igvc_description)/assets/part_21.stl"/>
+      </geometry>
+    </collision>
+    <!-- Part part_15 -->
+    <visual>
+      <origin xyz="-0.193704 -0.552769 0.227447" rpy="0 0 0"/>
+      <geometry>
+        <mesh filename="file://$(find igvc_description)/assets/part_15.stl"/>
+      </geometry>
+      <material name="part_15_material">
+        <color rgba="0.647059 0.647059 0.647059 1"/>
+      </material>
+    </visual>
+    <collision>
+      <origin xyz="-0.193704 -0.552769 0.227447" rpy="0 0 0"/>
+      <geometry>
+        <mesh filename="file://$(find igvc_description)/assets/part_15.stl"/>
+      </geometry>
+    </collision>
+    <!-- Part part_17_2 -->
+    <visual>
+      <origin xyz="0.0837819 -0.387669 0.441433" rpy="-1.5708 0 0"/>
+      <geometry>
+        <mesh filename="file://$(find igvc_description)/assets/part_17.stl"/>
+      </geometry>
+      <material name="part_17_2_material">
+        <color rgba="0.647059 0.647059 0.647059 1"/>
+      </material>
+    </visual>
+    <collision>
+      <origin xyz="0.0837819 -0.387669 0.441433" rpy="-1.5708 0 0"/>
+      <geometry>
+        <mesh filename="file://$(find igvc_description)/assets/part_17.stl"/>
+      </geometry>
+    </collision>
+    <!-- Part part_19 -->
+    <visual>
+      <origin xyz="-0.193704 -0.552769 0.227447" rpy="0 0 0"/>
+      <geometry>
+        <mesh filename="file://$(find igvc_description)/assets/part_19.stl"/>
+      </geometry>
+      <material name="part_19_material">
+        <color rgba="0.647059 0.647059 0.647059 1"/>
+      </material>
+    </visual>
+    <collision>
+      <origin xyz="-0.193704 -0.552769 0.227447" rpy="0 0 0"/>
+      <geometry>
+        <mesh filename="file://$(find igvc_description)/assets/part_19.stl"/>
+      </geometry>
+    </collision>
     <!-- Part part_5 -->
     <visual>
-      <origin xyz="0 -0.4572 -0.00635" rpy="0 -0 0"/>
+      <origin xyz="-0.193704 -0.552769 0.227447" rpy="0 0 0"/>
       <geometry>
         <mesh filename="file://$(find igvc_description)/assets/part_5.stl"/>
@@ -21,12 +357,124 @@
     </visual>
     <collision>
-      <origin xyz="0 -0.4572 -0.00635" rpy="0 -0 0"/>
+      <origin xyz="-0.193704 -0.552769 0.227447" rpy="0 0 0"/>
       <geometry>
         <mesh filename="file://$(find igvc_description)/assets/part_5.stl"/>
       </geometry>
     </collision>
+    <!-- Part part_17_3 -->
+    <visual>
+      <origin xyz="-0.193704 -0.552769 0.227447" rpy="0 0 0"/>
+      <geometry>
+        <mesh filename="file://$(find igvc_description)/assets/part_17.stl"/>
+      </geometry>
+      <material name="part_17_3_material">
+        <color rgba="0.647059 0.647059 0.647059 1"/>
+      </material>
+    </visual>
+    <collision>
+      <origin xyz="-0.193704 -0.552769 0.227447" rpy="0 0 0"/>
+      <geometry>
+        <mesh filename="file://$(find igvc_description)/assets/part_17.stl"/>
+      </geometry>
+    </collision>
+    <!-- Part part_18 -->
+    <visual>
+      <origin xyz="-0.193704 -0.552769 0.227447" rpy="0 0 0"/>
+      <geometry>
+        <mesh filename="file://$(find igvc_description)/assets/part_18.stl"/>
+      </geometry>
+      <material name="part_18_material">
+        <color rgba="0.647059 0.647059 0.647059 1"/>
+      </material>
+    </visual>
+    <collision>
+      <origin xyz="-0.193704 -0.552769 0.227447" rpy="0 0 0"/>
+      <geometry>
+        <mesh filename="file://$(find igvc_description)/assets/part_18.stl"/>
+      </geometry>
+    </collision>
+    <!-- Part part_32 -->
+    <visual>
+      <origin xyz="-0.193704 -0.552769 0.227447" rpy="0 0 0"/>
+      <geometry>
+        <mesh filename="file://$(find igvc_description)/assets/part_32.stl"/>
+      </geometry>
+      <material name="part_32_material">
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
Commit message: Almost running, controller manager dying on launch

File: src/igvc_description/urdf/model.urdf.xacro (robot description, xacro)
@@ -164,5 +164,5 @@
   </link>
   <!-- Joint from part_1 to part_10 -->
-  <joint name="wheel_L" type="continuous">
+  <joint name="left_wheel_joint" type="continuous">
     <origin xyz="-0.2159 0 -0.01905" rpy="1.5708 -0 1.5708"/>
     <parent link="part_1"/>
@@ -196,5 +196,5 @@
   </link>
   <!-- Joint from part_1 to part_9 -->
-  <joint name="wheel_R" type="continuous">
+  <joint name="right_wheel_joint" type="continuous">
     <origin xyz="0.2159 0 -0.01905" rpy="-1.5708 -0 1.5708"/>
     <parent link="part_1"/>
