Commit message: Updated the robot CAD and added material values.

File: src/igvc_description/urdf/model.urdf.xacro (robot description, xacro)
@@ -1,32 +1,192 @@
 <?xml version="1.0" ?>
 <!-- Generated using onshape-to-robot -->
-<!-- Onshape https://cad.onshape.com/documents/bd8c1cbb3cbd66454183450f/w/dfd94c9f83ff0fc6c8761109/e/b8893f818205c61a56339f3e -->
-<robot xmlns:xacro="http://www.ros.org/wiki/xacro">
+<!-- Onshape https://cad.onshape.com/documents/4f27315f66a4121bf8434c1a/w/bce24b18b959f9c2227327f4/e/534f540c791514c4a2b9f32e -->
+<robot name="igvc_description">
   <!-- Link part_1 -->
   <link name="part_1">
     <inertial>
-      <origin xyz="0 0 0" rpy="0 0 0"/>
-      <mass value="1e-03"/>
-      <inertia ixx="1e-03" ixy="0" ixz="0" iyy="1e-03" iyz="0" izz="1e-03"/>
+      <origin xyz="-0.0368571 0.291615 0.214315" rpy="0 0 0"/>
+      <mass value="56.0674"/>
+      <inertia ixx="3.60749" ixy="0" ixz="0" iyy="1.28472" iyz="0.159952" izz="3.84124"/>
     </inertial>
-    <!-- Part part_22 -->
-    <visual>
-      <origin xyz="-0.193704 -0.552769 0.227447" rpy="0 0 0"/>
-      <geometry>
-        <mesh filename="file://$(find igvc_description)/assets/part_22.stl"/>
-      </geometry>
-      <material name="part_22_material">
-        <color rgba="0.647059 0.647059 0.647059 1"/>
-      </material>
-    </visual>
-    <collision>
-      <origin xyz="-0.193704 -0.552769 0.227447" rpy="0 0 0"/>
-      <geometry>
-        <mesh filename="file://$(find igvc_description)/assets/part_22.stl"/>
+    <!-- Part part_9 -->
+    <visual>
+      <origin xyz="-0.0368571 -0.178453 0.142065" rpy="0 -0 0"/>
+      <geometry>
+        <mesh filename="file://$(find igvc_description)/assets/part_9.stl"/>
+      </geometry>
+      <material name="part_9_material">
+        <color rgba="0.647059 0.647059 0.647059 1"/>
+      </material>
+    </visual>
+    <collision>
+      <origin xyz="-0.0368571 -0.178453 0.142065" rpy="0 -0 0"/>
+      <geometry>
+        <mesh filename="file://$(find igvc_description)/assets/part_9.stl"/>
+      </geometry>
+    </collision>
+    <!-- Part part_33 -->
+    <visual>
+      <origin xyz="-0.0368571 -0.178453 0.142065" rpy="0 -0 0"/>
+      <geometry>
+        <mesh filename="file://$(find igvc_description)/assets/part_33.stl"/>
+      </geometry>
+      <material name="part_33_material">
+        <color rgba="1 0 0 1"/>
+      </material>
+    </visual>
+    <collision>
+      <origin xyz="-0.0368571 -0.178453 0.142065" rpy="0 -0 0"/>
+      <geometry>
+        <mesh filename="file://$(find igvc_description)/assets/part_33.stl"/>
+      </geometry>
+    </collision>
+    <!-- Part part_14 -->
+    <visual>
+      <origin xyz="-0.0368571 -0.178453 0.142065" rpy="0 -0 0"/>
+      <geometry>
+        <mesh filename="file://$(find igvc_description)/assets/part_14.stl"/>
+      </geometry>
+      <material name="part_14_material">
+        <color rgba="0.647059 0.647059 0.647059 1"/>
+      </material>
+    </visual>
+    <collision>
+      <origin xyz="-0.0368571 -0.178453 0.142065" rpy="0 -0 0"/>
+      <geometry>
+        <mesh filename="file://$(find igvc_description)/assets/part_14.stl"/>
+      </geometry>
+    </collision>
+    <!-- Part part_23 -->
+    <visual>
+      <origin xyz="-0.0368571 -0.178453 0.142065" rpy="0 -0 0"/>
+      <geometry>
+        <mesh filename="file://$(find igvc_description)/assets/part_23.stl"/>
+      </geometry>
+      <material name="part_23_material">
+        <color rgba="0.647059 0.647059 0.647059 1"/>
+      </material>
+    </visual>
+    <collision>
+      <origin xyz="-0.0368571 -0.178453 0.142065" rpy="0 -0 0"/>
+      <geometry>
+        <mesh filename="file://$(find igvc_description)/assets/part_23.stl"/>
+      </geometry>
+    </collision>
+    <!-- Part part_5 -->
+    <visual>
+      <origin xyz="-0.0368571 -0.178453 0.142065" rpy="0 -0 0"/>
+      <geometry>
+        <mesh filename="file://$(find igvc_description)/assets/part_5.stl"/>
+      </geometry>
+      <material name="part_5_material">
+        <color rgba="0.647059 0.647059 0.647059 1"/>
+      </material>
+    </visual>
+    <collision>
+      <origin xyz="-0.0368571 -0.178453 0.142065" rpy="0 -0 0"/>
+      <geometry>
+        <mesh filename="file://$(find igvc_description)/assets/part_5.stl"/>
+      </geometry>
+    </collision>
+    <!-- Part part_1 -->
+    <visual>
+      <origin xyz="-0.0368571 -0.178453 0.142065" rpy="0 -0 0"/>
+      <geometry>
+        <mesh filename="file://$(find igvc_description)/assets/part_1.stl"/>
+      </geometry>
+      <material name="part_1_material">
+        <color rgba="0.647059 0.647059 0.647059 1"/>
+      </material>
+    </visual>
+    <collision>
+      <origin xyz="-0.0368571 -0.178453 0.142065" rpy="0 -0 0"/>
+      <geometry>
+        <mesh filename="file://$(find igvc_description)/assets/part_1.stl"/>
+      </geometry>
+    </collision>
+    <!-- Part part_28 -->
+    <visual>
+      <origin xyz="-0.0368571 -0.178453 0.142065" rpy="0 -0 0"/>
+      <geometry>
+        <mesh filename="file://$(find igvc_description)/assets/part_28.stl"/>
+      </geometry>
+      <material name="part_28_material">
+        <color rgba="0.941176 0.87451 0.678431 1"/>
+      </material>
+    </visual>
+    <collision>
+      <origin xyz="-0.0368571 -0.178453 0.142065" rpy="0 -0 0"/>
+      <geometry>
+        <mesh filename="file://$(find igvc_description)/assets/part_28.stl"/>
+      </geometry>
+    </collision>
+    <!-- Part part_12 -->
+    <visual>
+      <origin xyz="-0.0368571 -0.178453 0.142065" rpy="0 -0 0"/>
+      <geometry>
+        <mesh filename="file://$(find igvc_description)/assets/part_12.stl"/>
+      </geometry>
+      <material name="part_12_material">
+        <color rgba="0.647059 0.647059 0.647059 1"/>
+      </material>
+    </visual>
+    <collision>
+      <origin xyz="-0.0368571 -0.178453 0.142065" rpy="0 -0 0"/>
+      <geometry>
+        <mesh filename="file://$(find igvc_description)/assets/part_12.stl"/>
+      </geometry>
+    </collision>
+    <!-- Part part_30 -->
+    <visual>
+      <origin xyz="-0.0368571 -0.178453 0.142065" rpy="0 -0 0"/>
+      <geometry>
+        <mesh filename="file://$(find igvc_description)/assets/part_30.stl"/>
+      </geometry>
+      <material name="part_30_material">
+        <color rgba="0.286275 0.266667 0.266667 1"/>
+      </material>
+    </visual>
+    <collision>
+      <origin xyz="-0.0368571 -0.178453 0.142065" rpy="0 -0 0"/>
+      <geometry>
+        <mesh filename="file://$(find igvc_description)/assets/part_30.stl"/>
+      </geometry>
+    </collision>
+    <!-- Part part_39 -->
+    <visual>
+      <origin xyz="-0.0368571 -0.178453 0.142065" rpy="0 -0 0"/>
+      <geometry>
+        <mesh filename="file://$(find igvc_description)/assets/part_39.stl"/>
+      </geometry>
+      <material name="part_39_material">
+        <color rgba="0.286275 0.266667 0.266667 1"/>
+      </material>
+    </visual>
+    <collision>
+      <origin xyz="-0.0368571 -0.178453 0.142065" rpy="0 -0 0"/>
+      <geometry>
+        <mesh filename="file://$(find igvc_description)/assets/part_39.stl"/>
+      </geometry>
+    </collision>
+    <!-- Part part_19 -->
+    <visual>
+      <origin xyz="-0.0368571 -0.178453 0.142065" rpy="0 -0 0"/>
+      <geometry>
+        <mesh filename="file://$(find igvc_description)/assets/part_19.stl"/>
+      </geometry>
+      <material name="part_19_material">
+        <color rgba="0.647059 0.647059 0.647059 1"/>
+      </material>
+    </visual>
+    <collision>
+      <origin xyz="-0.0368571 -0.178453 0.142065" rpy="0 -0 0"/>
+      <geometry>
+        <mesh filename="file://$(find igvc_description)/assets/part_19.stl"/>
       </geometry>
     </collision>
     <!-- Part part_3 -->
     <visual>
-      <origin xyz="-0.193704 -0.552769 0.227447" rpy="0 0 0"/>
+      <origin xyz="-0.0368571 -0.178453 0.142065" rpy="0 -0 0"/>
       <geometry>
         <mesh filename="file://$(find igvc_description)/assets/part_3.stl"/>
@@ -37,28 +197,28 @@
     </visual>
     <collision>
-      <origin xyz="-0.193704 -0.552769 0.227447" rpy="0 0 0"/>
+      <origin xyz="-0.0368571 -0.178453 0.142065" rpy="0 -0 0"/>
       <geometry>
         <mesh filename="file://$(find igvc_description)/assets/part_3.stl"/>
       </geometry>
     </collision>
-    <!-- Part part_17 -->
-    <visual>
-      <origin xyz="0.0837819 0.221931 0.441433" rpy="-1.5708 -0 -0"/>
-      <geometry>
-        <mesh filename="file://$(find igvc_description)/assets/part_17.stl"/>
-      </geometry>
-      <material name="part_17_material">
-        <color rgba="0.647059 0.647059 0.647059 1"/>
-      </material>
-    </visual>
-    <collision>
-      <origin xyz="0.0837819 0.221931 0.441433" rpy="-1.5708 -0 -0"/>
-      <geometry>
-        <mesh filename="file://$(find igvc_description)/assets/part_17.stl"/>
+    <!-- Part part_32 -->
+    <visual>
+      <origin xyz="-0.0368571 -0.178453 0.142065" rpy="0 -0 0"/>
+      <geometry>
+        <mesh filename="file://$(find igvc_description)/assets/part_32.stl"/>
+      </geometry>
+      <material name="part_32_material">
+        <color rgba="0.647059 0.647059 0.647059 1"/>
+      </material>
+    </visual>
+    <collision>
+      <origin xyz="-0.0368571 -0.178453 0.142065" rpy="0 -0 0"/>
+      <geometry>
+        <mesh filename="file://$(find igvc_description)/assets/part_32.stl"/>
       </geometry>
     </collision>
     <!-- Part part_27 -->
     <visual>
-      <origin xyz="-0.193704 -0.552769 0.227447" rpy="0 0 0"/>
+      <origin xyz="-0.0368571 -0.178453 0.142065" rpy="0 -0 0"/>
       <geometry>
         <mesh filename="file://$(find igvc_description)/assets/part_27.stl"/>
@@ -69,12 +229,268 @@
     </visual>
     <collision>
-      <origin xyz="-0.193704 -0.552769 0.227447" rpy="0 0 0"/>
+      <origin xyz="-0.0368571 -0.178453 0.142065" rpy="0 -0 0"/>
       <geometry>
         <mesh filename="file://$(find igvc_description)/assets/part_27.stl"/>
       </geometry>
     </collision>
+    <!-- Part part_22 -->
+    <visual>
+      <origin xyz="-0.0368571 -0.178453 0.142065" rpy="0 -0 0"/>
+      <geometry>
+        <mesh filename="file://$(find igvc_description)/assets/part_22.stl"/>
+      </geometry>
+      <material name="part_22_material">
+        <color rgba="0.647059 0.647059 0.647059 1"/>
+      </material>
+    </visual>
+    <collision>
+      <origin xyz="-0.0368571 -0.178453 0.142065" rpy="0 -0 0"/>
+      <geometry>
+        <mesh filename="file://$(find igvc_description)/assets/part_22.stl"/>
+      </geometry>
+    </collision>
+    <!-- Part part_13 -->
+    <visual>
+      <origin xyz="-0.0368571 -0.178453 0.142065" rpy="0 -0 0"/>
+      <geometry>
+        <mesh filename="file://$(find igvc_description)/assets/part_13.stl"/>
+      </geometry>
+      <material name="part_13_material">
+        <color rgba="0.647059 0.647059 0.647059 1"/>
+      </material>
+    </visual>
+    <collision>
+      <origin xyz="-0.0368571 -0.178453 0.142065" rpy="0 -0 0"/>
+      <geometry>
+        <mesh filename="file://$(find igvc_description)/assets/part_13.stl"/>
+      </geometry>
+    </collision>
+    <!-- Part part_16 -->
+    <visual>
+      <origin xyz="-0.0368571 -0.178453 0.142065" rpy="0 -0 0"/>
+      <geometry>
+        <mesh filename="file://$(find igvc_description)/assets/part_16.stl"/>
+      </geometry>
+      <material name="part_16_material">
+        <color rgba="0.647059 0.647059 0.647059 1"/>
+      </material>
+    </visual>
+    <collision>
+      <origin xyz="-0.0368571 -0.178453 0.142065" rpy="0 -0 0"/>
+      <geometry>
+        <mesh filename="file://$(find igvc_description)/assets/part_16.stl"/>
+      </geometry>
+    </collision>
+    <!-- Part part_7 -->
+    <visual>
+      <origin xyz="-0.0368571 -0.178453 0.142065" rpy="0 -0 0"/>
+      <geometry>
+        <mesh filename="file://$(find igvc_description)/assets/part_7.stl"/>
+      </geometry>
+      <material name="part_7_material">
+        <color rgba="0.647059 0.647059 0.647059 1"/>
+      </material>
+    </visual>
+    <collision>
+      <origin xyz="-0.0368571 -0.178453 0.142065" rpy="0 -0 0"/>
+      <geometry>
+        <mesh filename="file://$(find igvc_description)/assets/part_7.stl"/>
+      </geometry>
+    </collision>
+    <!-- Part part_21 -->
+    <visual>
+      <origin xyz="-0.0368571 -0.178453 0.142065" rpy="0 -0 0"/>
+      <geometry>
+        <mesh filename="file://$(find igvc_description)/assets/part_21.stl"/>
+      </geometry>
+      <material name="part_21_material">
+        <color rgba="0.647059 0.647059 0.647059 1"/>
+      </material>
+    </visual>
+    <collision>
+      <origin xyz="-0.0368571 -0.178453 0.142065" rpy="0 -0 0"/>
+      <geometry>
+        <mesh filename="file://$(find igvc_description)/assets/part_21.stl"/>
+      </geometry>
+    </collision>
+    <!-- Part part_38 -->
+    <visual>
+      <origin xyz="-0.0368571 -0.178453 0.142065" rpy="0 -0 0"/>
+      <geometry>
+        <mesh filename="file://$(find igvc_description)/assets/part_38.stl"/>
+      </geometry>
+      <material name="part_38_material">
+        <color rgba="0.917647 0.917647 0.917647 1"/>
+      </material>
+    </visual>
+    <collision>
+      <origin xyz="-0.0368571 -0.178453 0.142065" rpy="0 -0 0"/>
+      <geometry>
+        <mesh filename="file://$(find igvc_description)/assets/part_38.stl"/>
+      </geometry>
+    </collision>
+    <!-- Part part_4 -->
+    <visual>
+      <origin xyz="-0.0368571 -0.178453 0.142065" rpy="0 -0 0"/>
+      <geometry>
+        <mesh filename="file://$(find igvc_description)/assets/part_4.stl"/>
+      </geometry>
+      <material name="part_4_material">
+        <color rgba="0.647059 0.647059 0.647059 1"/>
+      </material>
+    </visual>
+    <collision>
+      <origin xyz="-0.0368571 -0.178453 0.142065" rpy="0 -0 0"/>
+      <geometry>
+        <mesh filename="file://$(find igvc_description)/assets/part_4.stl"/>
+      </geometry>
+    </collision>
+    <!-- Part part_18 -->
+    <visual>
+      <origin xyz="-0.0368571 -0.178453 0.142065" rpy="0 -0 0"/>
+      <geometry>
+        <mesh filename="file://$(find igvc_description)/assets/part_18.stl"/>
+      </geometry>
+      <material name="part_18_material">
+        <color rgba="0.647059 0.647059 0.647059 1"/>
+      </material>
+    </visual>
+    <collision>
+      <origin xyz="-0.0368571 -0.178453 0.142065" rpy="0 -0 0"/>
+      <geometry>
+        <mesh filename="file://$(find igvc_description)/assets/part_18.stl"/>
+      </geometry>
+    </collision>
+    <!-- Part part_24 -->
+    <visual>
+      <origin xyz="-0.0368571 -0.178453 0.142065" rpy="0 -0 0"/>
+      <geometry>
+        <mesh filename="file://$(find igvc_description)/assets/part_24.stl"/>
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
Commit message: partially working drive simulation

File: src/igvc_description/urdf/model.urdf.xacro (robot description, xacro)
@@ -7,6 +7,6 @@
     <inertial>
       <origin xyz="0 0 0" rpy="0 0 0"/>
-      <mass value="1e-03"/>
-      <inertia ixx="1e-03" ixy="0" ixz="0" iyy="1e-03" iyz="0" izz="1e-03"/>
+      <mass value="1"/>
+      <inertia ixx="1" ixy="0" ixz="0" iyy="1" iyz="0" izz="1"/>
     </inertial>
     <!-- Part part_5 -->
@@ -143,6 +143,6 @@
     <inertial>
       <origin xyz="0 0 0" rpy="0 0 0"/>
-      <mass value="1e-03"/>
-      <inertia ixx="1e-03" ixy="0" ixz="0" iyy="1e-03" iyz="0" izz="1e-03"/>
+      <mass value="1"/>
+      <inertia ixx="1" ixy="0" ixz="0" iyy="1" iyz="0" izz="1"/>
     </inertial>
     <!-- Part part_10 -->
@@ -175,6 +175,6 @@
     <inertial>
       <origin xyz="0 0 0" rpy="0 0 0"/>
-      <mass value="1e-03"/>
-      <inertia ixx="1e-03" ixy="0" ixz="0" iyy="1e-03" iyz="0" izz="1e-03"/>
+      <mass value="1"/>
+      <inertia ixx="1" ixy="0" ixz="0" iyy="1" iyz="0" izz="1"/>
     </inertial>
     <!-- Part part_9 -->

File: src/igvc_description/urdf/robot.urdf.xacro (robot description, xacro)
@@ -14,3 +14,8 @@
     <xacro:include filename="$(find igvc_hardware)/description/bot.ros2_control.xacro" />
     <xacro:bot_ros2_control name="IGVC_Bot" prefix="$(arg prefix)" use_mock_hardware="$(arg use_mock_hardware)"/>
+    <gazebo>
+        <plugin filename="gz_ros2_control-system" name="gz_ros2_control::GazeboSimROS2ControlPlugin">
+        <parameters>$(find igvc_hardware)/config/bot_controllers.yaml</parameters>
+        </plugin>
+    </gazebo>
 </robot>

File: src/igvc_hardware/description/bot.ros2_control.xacro (robot description, xacro)
@@ -13,6 +13,5 @@
       <xacro:if value="${use_mock_hardware}">
         <hardware>
-          <plugin>mock_components/GenericSystem</plugin>
-          <param name="calculate_dynamics">true</param>
+          <plugin>gz_ros2_control/GazeboSimSystem</plugin>
         </hardware>
       </xacro:if>
