Commit message: Updated URDF V1  (#15)
* Transition Hardware package to igvc_hardware

* Create nav, gazebo, slam packages

* Create description package

* Modify igvc_description CMakeLists

* Add oak description to decription package

* Remove placeholder uml

* implement navigation package

* Implement slam package, TODO tune for igvc

* Remove redundant CMake library targets

* Generate low fidelity sim model URDF

* Add onshape-to-robot config file

* Rename otr urdf to model

* Create robot urdf file

* Add rviz launch files

* Change hardware package name to igvc_hardware

* Correct project name in slam package cmakelist

* Correct meshes to assets in description cmake

* Remove references to deprecated urdf file

* add package name to URDF meshes (automate this in the future)

* Remove nonexistent adi rosdep

* Remove nonexistent odrive rosdep

* Add gz and gz control plugin to gazebo dependencies

* Add directories to gazebo cmake

* Implement empty world files

* Rename robot in launch file

* Placeholder sensor simulation and bridge configuration

* Add config directory to gazebo cmake

* Split rviz and publisher into separate launches

* Include publisher launch file in gazebo launch

* Remove unused imports

* Configure RGBD camera description

* Remove madgwick filter from sim launch file

* rename launch file to hardware.launch.py

* Update hardware bringups to have the proper ODrive drivetrain

* Add IMU node to hardware launch

* rename hardware xacro

* Add hardware xacro to robot xacro

* remove joint state broadcaster from controllers yaml

* Update src/igvc_gazebo/launch/empty_world.launch.py

Co-authored-by: Mathew Davis <mjdavis0504@gmail.com>

* Update src/igvc_gazebo/launch/empty_world.launch.py

Co-authored-by: Mathew Davis <mjdavis0504@gmail.com>

* Fix file URDF locations

* Reconfigure robot description to use hardware package for ros2 control

* Remove duplicate OAK and position existing camera

* Change oak name, add igvc_robot to sensor xacro

* Fix devcontainer symlink install

* add friction to ground plane

* Change sensor formatting to recommended format

* Update bridge topic names

* Alter inertial values

* Change robot spawn location

* Reconfigure OAK simulation URDF

* Change rtabmap sim launch

* Update URDF to Low Fidelity V1

* Updated the robot CAD and added material values.

* Transition Hardware package to igvc_hardware

* Create nav, gazebo, slam packages

* Create description package

* Modify igvc_description CMakeLists

* Add oak description to decription package

* Remove placeholder uml

* implement navigation package

* Implement slam package, TODO tune for igvc

* Remove redundant CMake library targets

* Generate low fidelity sim model URDF

* Rename otr urdf to model

* Create robot urdf file

* Add rviz launch files

* Correct project name in slam package cmakelist

* Correct meshes to assets in description cmake

* Remove references to deprecated urdf file

* add package name to URDF meshes (automate this in the future)

* Add gz and gz control plugin to gazebo dependencies

* Add directories to gazebo cmake

* Implement empty world files

* Rename robot in launch file

* Placeholder sensor simulation and bridge configuration

* Add config directory to gazebo cmake

* Split rviz and publisher into separate launches

* Include publisher launch file in gazebo launch

* Remove unused imports

* Configure RGBD camera description

* Remove madgwick filter from sim launch file

* rename launch file to hardware.launch.py

* Update hardware bringups to have the proper ODrive drivetrain

* Add IMU node to hardware launch

* rename hardware xacro

* Add hardware xacro to robot xacro

* Update src/igvc_gazebo/launch/empty_world.launch.py

Co-authored-by: Mathew Davis <mjdavis0504@gmail.com>

* Update src/igvc_gazebo/launch/empty_world.launch.py

Co-authored-by: Mathew Davis <mjdavis0504@gmail.com>

* Fix file URDF locations

* Reconfigure robot description to use hardware package for ros2 control

* Remove duplicate OAK and position existing camera

* Change oak name, add igvc_robot to sensor xacro

* add friction to ground plane

* Change sensor formatting to recommended format

* Update bridge topic names

* Alter inertial values

* Change robot spawn location

* Reconfigure OAK simulation URDF

* Change rtabmap sim launch

* Update URDF to Low Fidelity V1

* Updated the robot CAD and added material values.

* Remove model.txt

* Remove publisher launch from rtabmap launch

* Remove unnecessary exports

* Fix naming reversions

* Revert gazebo and nav2 naming changes

---------

Co-authored-by: Zane Brotherton <zanebrotherton@gmail.com>
Co-authored-by: tagciccone <tagciccone@gmail.com>
Co-authored-by: Zane Brotherton <46907447+zbrotherton@users.noreply.github.com>
Co-authored-by: Tag Ciccone <109768604+TagCiccone@users.noreply.github.com>

File: src/igvc_description/urdf/model.urdf.xacro (robot description, xacro)
@@ -1,205 +1,717 @@
 <?xml version="1.0" ?>
 <!-- Generated using onshape-to-robot -->
-<!-- Onshape https://cad.onshape.com/documents/bd8c1cbb3cbd66454183450f/w/dfd94c9f83ff0fc6c8761109/e/c765fc0d53504544c054bc0a -->
-<robot xmlns:xacro="http://www.ros.org/wiki/xacro">
+<!-- Onshape https://cad.onshape.com/documents/4f27315f66a4121bf8434c1a/w/bce24b18b959f9c2227327f4/e/534f540c791514c4a2b9f32e -->
+<robot name="igvc_description">
   <!-- Link part_1 -->
   <link name="part_1">
     <inertial>
-      <origin xyz="0 0 0" rpy="0 0 0"/>
-      <mass value="1e-03"/>
-      <inertia ixx="1e-03" ixy="0" ixz="0" iyy="1e-03" iyz="0" izz="1e-03"/>
-    </inertial>
-    <!-- Part part_5 -->
-    <visual>
-      <origin xyz="0 -0.4572 -0.00635" rpy="0 -0 0"/>
-      <geometry>
-        <mesh filename="file://$(find igvc_description)/assets/part_5.stl"/>
-      </geometry>
-      <material name="part_5_material">
-        <color rgba="0.647059 0.647059 0.647059 1"/>
-      </material>
-    </visual>
-    <collision>
-      <origin xyz="0 -0.4572 -0.00635" rpy="0 -0 0"/>
-      <geometry>
-        <mesh filename="file://$(find igvc_description)/assets/part_5.stl"/>
-      </geometry>
-    </collision>
-    <!-- Part part_4 -->
-    <visual>
-      <origin xyz="0 -0.4572 -0.00635" rpy="0 -0 0"/>
-      <geometry>
-        <mesh filename="file://$(find igvc_description)/assets/part_4.stl"/>
-      </geometry>
-      <material name="part_4_material">
-        <color rgba="0.647059 0.647059 0.647059 1"/>
-      </material>
-    </visual>
-    <collision>
-      <origin xyz="0 -0.4572 -0.00635" rpy="0 -0 0"/>
-      <geometry>
-        <mesh filename="file://$(find igvc_description)/assets/part_4.stl"/>
-      </geometry>
-    </collision>
-    <!-- Part part_8 -->
-    <visual>
-      <origin xyz="0 -0.4572 -0.00635" rpy="0 -0 0"/>
-      <geometry>
-        <mesh filename="file://$(find igvc_description)/assets/part_8.stl"/>
-      </geometry>
-      <material name="part_8_material">
-        <color rgba="0.647059 0.647059 0.647059 1"/>
-      </material>
-    </visual>
-    <collision>
-      <origin xyz="0 -0.4572 -0.00635" rpy="0 -0 0"/>
-      <geometry>
-        <mesh filename="file://$(find igvc_description)/assets/part_8.stl"/>
-      </geometry>
-    </collision>
-    <!-- Part part_2 -->
-    <visual>
-      <origin xyz="0 -0.4572 -0.00635" rpy="0 -0 0"/>
-      <geometry>
-        <mesh filename="file://$(find igvc_description)/assets/part_2.stl"/>
-      </geometry>
-      <material name="part_2_material">
-        <color rgba="0.647059 0.647059 0.647059 1"/>
-      </material>
-    </visual>
-    <collision>
-      <origin xyz="0 -0.4572 -0.00635" rpy="0 -0 0"/>
-      <geometry>
-        <mesh filename="file://$(find igvc_description)/assets/part_2.stl"/>
-      </geometry>
-    </collision>
-    <!-- Part part_6 -->
-    <visual>
-      <origin xyz="0 -0.4572 -0.00635" rpy="0 -0 0"/>
-      <geometry>
-        <mesh filename="file://$(find igvc_description)/assets/part_6.stl"/>
-      </geometry>
-      <material name="part_6_material">
-        <color rgba="0.231373 0.380392 0.705882 1"/>
-      </material>
-    </visual>
-    <collision>
-      <origin xyz="0 -0.4572 -0.00635" rpy="0 -0 0"/>
-      <geometry>
-        <mesh filename="file://$(find igvc_description)/assets/part_6.stl"/>
-      </geometry>
-    </collision>
-    <!-- Part part_3 -->
-    <visual>
-      <origin xyz="0 -0.4572 -0.00635" rpy="0 -0 0"/>
-      <geometry>
-        <mesh filename="file://$(find igvc_description)/assets/part_3.stl"/>
-      </geometry>
-      <material name="part_3_material">
-        <color rgba="0.647059 0.647059 0.647059 1"/>
-      </material>
-    </visual>
-    <collision>
-      <origin xyz="0 -0.4572 -0.00635" rpy="0 -0 0"/>
-      <geometry>
-        <mesh filename="file://$(find igvc_description)/assets/part_3.stl"/>
-      </geometry>
-    </collision>
-    <!-- Part part_7 -->
-    <visual>
-      <origin xyz="0 -0.4572 -0.00635" rpy="0 -0 0"/>
-      <geometry>
-        <mesh filename="file://$(find igvc_description)/assets/part_7.stl"/>
-      </geometry>
-      <material name="part_7_material">
-        <color rgba="0.498039 0.498039 0.498039 1"/>
-      </material>
-    </visual>
-    <collision>
-      <origin xyz="0 -0.4572 -0.00635" rpy="0 -0 0"/>
-      <geometry>
-        <mesh filename="file://$(find igvc_description)/assets/part_7.stl"/>
-      </geometry>
-    </collision>
-    <!-- Part part_1 -->
-    <visual>
-      <origin xyz="0 -0.4572 -0.00635" rpy="0 -0 0"/>
-      <geometry>
-        <mesh filename="file://$(find igvc_description)/assets/part_1.stl"/>
-      </geometry>
-      <material name="part_1_material">
-        <color rgba="0.647059 0.647059 0.647059 1"/>
-      </material>
-    </visual>
-    <collision>
-      <origin xyz="0 -0.4572 -0.00635" rpy="0 -0 0"/>
-      <geometry>
-        <mesh filename="file://$(find igvc_description)/assets/part_1.stl"/>
-      </geometry>
-    </collision>
-  </link>
-  <!-- Link part_10 -->
-  <link name="part_10">
-    <inertial>
-      <origin xyz="0 0 0" rpy="0 0 0"/>
-      <mass value="1e-03"/>
-      <inertia ixx="1e-03" ixy="0" ixz="0" iyy="1e-03" iyz="0" izz="1e-03"/>
-    </inertial>
-    <!-- Part part_10 -->
-    <visual>
-      <origin xyz="-0.4572 -0 0.2159" rpy="-1.5708 -1.5708 0"/>
-      <geometry>
-        <mesh filename="file://$(find igvc_description)/assets/part_10.stl"/>
-      </geometry>
-      <material name="part_10_material">
-        <color rgba="0.286275 0.266667 0.266667 1"/>
-      </material>
-    </visual>
-    <collision>
-      <origin xyz="-0.4572 -0 0.2159" rpy="-1.5708 -1.5708 0"/>
-      <geometry>
-        <mesh filename="file://$(find igvc_description)/assets/part_10.stl"/>
-      </geometry>
-    </collision>
-  </link>
-  <!-- Joint from part_1 to part_10 -->
-  <joint name="wheel_L" type="continuous">
-    <origin xyz="-0.2159 0 -0.01905" rpy="1.5708 -0 1.5708"/>
-    <parent link="part_1"/>
-    <child link="part_10"/>
-    <axis xyz="0 0 1"/>
-    <limit effort="10" velocity="10"/>
-  </joint>
-  <!-- Link part_9 -->
-  <link name="part_9">
-    <inertial>
-      <origin xyz="0 0 0" rpy="0 0 0"/>
-      <mass value="1e-03"/>
-      <inertia ixx="1e-03" ixy="0" ixz="0" iyy="1e-03" iyz="0" izz="1e-03"/>
+      <origin xyz="-0.0368571 0.291615 0.214315" rpy="0 0 0"/>
+      <mass value="56.0674"/>
+      <inertia ixx="3.60749" ixy="0" ixz="0" iyy="1.28472" iyz="0.159952" izz="3.84124"/>
     </inertial>
     <!-- Part part_9 -->
     <visual>
-      <origin xyz="-0.4572 0 0.2159" rpy="1.5708 1.5708 0"/>
+      <origin xyz="-0.0368571 -0.178453 0.142065" rpy="0 -0 0"/>
       <geometry>
         <mesh filename="file://$(find igvc_description)/assets/part_9.stl"/>
       </geometry>
       <material name="part_9_material">
+        <color rgba="0.647059 0.647059 0.647059 1"/>
+      </material>
+    </visual>
+    <collision>
+      <origin xyz="-0.0368571 -0.178453 0.142065" rpy="0 -0 0"/>
+      <geometry>
+        <mesh filename="file://$(find igvc_description)/assets/part_9.stl"/>
+      </geometry>
+    </collision>
+    <!-- Part part_33 -->
+    <visual>
+      <origin xyz="-0.0368571 -0.178453 0.142065" rpy="0 -0 0"/>
+      <geometry>
+        <mesh filename="file://$(find igvc_description)/assets/part_33.stl"/>
+      </geometry>
+      <material name="part_33_material">
+        <color rgba="1 0 0 1"/>
+      </material>
+    </visual>
+    <collision>
+      <origin xyz="-0.0368571 -0.178453 0.142065" rpy="0 -0 0"/>
+      <geometry>
+        <mesh filename="file://$(find igvc_description)/assets/part_33.stl"/>
+      </geometry>
+    </collision>
+    <!-- Part part_14 -->
+    <visual>
+      <origin xyz="-0.0368571 -0.178453 0.142065" rpy="0 -0 0"/>
+      <geometry>
+        <mesh filename="file://$(find igvc_description)/assets/part_14.stl"/>
+      </geometry>
+      <material name="part_14_material">
+        <color rgba="0.647059 0.647059 0.647059 1"/>
+      </material>
+    </visual>
+    <collision>
+      <origin xyz="-0.0368571 -0.178453 0.142065" rpy="0 -0 0"/>
+      <geometry>
+        <mesh filename="file://$(find igvc_description)/assets/part_14.stl"/>
+      </geometry>
+    </collision>
+    <!-- Part part_23 -->
+    <visual>
+      <origin xyz="-0.0368571 -0.178453 0.142065" rpy="0 -0 0"/>
+      <geometry>
+        <mesh filename="file://$(find igvc_description)/assets/part_23.stl"/>
+      </geometry>
+      <material name="part_23_material">
+        <color rgba="0.647059 0.647059 0.647059 1"/>
+      </material>
+    </visual>
+    <collision>
+      <origin xyz="-0.0368571 -0.178453 0.142065" rpy="0 -0 0"/>
+      <geometry>
+        <mesh filename="file://$(find igvc_description)/assets/part_23.stl"/>
+      </geometry>
+    </collision>
+    <!-- Part part_5 -->
+    <visual>
+      <origin xyz="-0.0368571 -0.178453 0.142065" rpy="0 -0 0"/>
+      <geometry>
+        <mesh filename="file://$(find igvc_description)/assets/part_5.stl"/>
+      </geometry>
+      <material name="part_5_material">
+        <color rgba="0.647059 0.647059 0.647059 1"/>
+      </material>
+    </visual>
+    <collision>
+      <origin xyz="-0.0368571 -0.178453 0.142065" rpy="0 -0 0"/>
+      <geometry>
+        <mesh filename="file://$(find igvc_description)/assets/part_5.stl"/>
+      </geometry>
+    </collision>
+    <!-- Part part_1 -->
+    <visual>
+      <origin xyz="-0.0368571 -0.178453 0.142065" rpy="0 -0 0"/>
+      <geometry>
+        <mesh filename="file://$(find igvc_description)/assets/part_1.stl"/>
+      </geometry>
+      <material name="part_1_material">
+        <color rgba="0.647059 0.647059 0.647059 1"/>
+      </material>
+    </visual>
+    <collision>
+      <origin xyz="-0.0368571 -0.178453 0.142065" rpy="0 -0 0"/>
+      <geometry>
+        <mesh filename="file://$(find igvc_description)/assets/part_1.stl"/>
+      </geometry>
+    </collision>
+    <!-- Part part_28 -->
+    <visual>
+      <origin xyz="-0.0368571 -0.178453 0.142065" rpy="0 -0 0"/>
+      <geometry>
+        <mesh filename="file://$(find igvc_description)/assets/part_28.stl"/>
+      </geometry>
+      <material name="part_28_material">
+        <color rgba="0.941176 0.87451 0.678431 1"/>
+      </material>
+    </visual>
+    <collision>
+      <origin xyz="-0.0368571 -0.178453 0.142065" rpy="0 -0 0"/>
+      <geometry>
+        <mesh filename="file://$(find igvc_description)/assets/part_28.stl"/>
+      </geometry>
+    </collision>
+    <!-- Part part_12 -->
+    <visual>
+      <origin xyz="-0.0368571 -0.178453 0.142065" rpy="0 -0 0"/>
+      <geometry>
+        <mesh filename="file://$(find igvc_description)/assets/part_12.stl"/>
+      </geometry>
+      <material name="part_12_material">
+        <color rgba="0.647059 0.647059 0.647059 1"/>
+      </material>
+    </visual>
+    <collision>
+      <origin xyz="-0.0368571 -0.178453 0.142065" rpy="0 -0 0"/>
+      <geometry>
+        <mesh filename="file://$(find igvc_description)/assets/part_12.stl"/>
+      </geometry>
+    </collision>
+    <!-- Part part_30 -->
+    <visual>
+      <origin xyz="-0.0368571 -0.178453 0.142065" rpy="0 -0 0"/>
+      <geometry>
+        <mesh filename="file://$(find igvc_description)/assets/part_30.stl"/>
+      </geometry>
+      <material name="part_30_material">
         <color rgba="0.286275 0.266667 0.266667 1"/>
       </material>
     </visual>
     <collision>
-      <origin xyz="-0.4572 0 0.2159" rpy="1.5708 1.5708 0"/>
-      <geometry>
-        <mesh filename="file://$(find igvc_description)/assets/part_9.stl"/>
+      <origin xyz="-0.0368571 -0.178453 0.142065" rpy="0 -0 0"/>
+      <geometry>
+        <mesh filename="file://$(find igvc_description)/assets/part_30.stl"/>
+      </geometry>
+    </collision>
+    <!-- Part part_39 -->
+    <visual>
+      <origin xyz="-0.0368571 -0.178453 0.142065" rpy="0 -0 0"/>
+      <geometry>
+        <mesh filename="file://$(find igvc_description)/assets/part_39.stl"/>
+      </geometry>
+      <material name="part_39_material">
+        <color rgba="0.286275 0.266667 0.266667 1"/>
+      </material>
+    </visual>
+    <collision>
+      <origin xyz="-0.0368571 -0.178453 0.142065" rpy="0 -0 0"/>
+      <geometry>
+        <mesh filename="file://$(find igvc_description)/assets/part_39.stl"/>
+      </geometry>
+    </collision>
+    <!-- Part part_19 -->
+    <visual>
+      <origin xyz="-0.0368571 -0.178453 0.142065" rpy="0 -0 0"/>
+      <geometry>
+        <mesh filename="file://$(find igvc_description)/assets/part_19.stl"/>
+      </geometry>
+      <material name="part_19_material">
+        <color rgba="0.647059 0.647059 0.647059 1"/>
+      </material>
+    </visual>
+    <collision>
+      <origin xyz="-0.0368571 -0.178453 0.142065" rpy="0 -0 0"/>
+      <geometry>
+        <mesh filename="file://$(find igvc_description)/assets/part_19.stl"/>
+      </geometry>
+    </collision>
+    <!-- Part part_3 -->
+    <visual>
+      <origin xyz="-0.0368571 -0.178453 0.142065" rpy="0 -0 0"/>
+      <geometry>
+        <mesh filename="file://$(find igvc_description)/assets/part_3.stl"/>
+      </geometry>
+      <material name="part_3_material">
+        <color rgba="0.647059 0.647059 0.647059 1"/>
+      </material>
+    </visual>
+    <collision>
+      <origin xyz="-0.0368571 -0.178453 0.142065" rpy="0 -0 0"/>
+      <geometry>
+        <mesh filename="file://$(find igvc_description)/assets/part_3.stl"/>
+      </geometry>
+    </collision>
+    <!-- Part part_32 -->
+    <visual>
+      <origin xyz="-0.0368571 -0.178453 0.142065" rpy="0 -0 0"/>
+      <geometry>
+        <mesh filename="file://$(find igvc_description)/assets/part_32.stl"/>
+      </geometry>
+      <material name="part_32_material">
+        <color rgba="0.647059 0.647059 0.647059 1"/>
+      </material>
+    </visual>
+    <collision>
+      <origin xyz="-0.0368571 -0.178453 0.142065" rpy="0 -0 0"/>
+      <geometry>
+        <mesh filename="file://$(find igvc_description)/assets/part_32.stl"/>
+      </geometry>
+    </collision>
+    <!-- Part part_27 -->
+    <visual>
+      <origin xyz="-0.0368571 -0.178453 0.142065" rpy="0 -0 0"/>
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
Commit message: Rename misnamed joints

File: src/igvc_description/urdf/model.urdf.xacro (robot description, xacro)
@@ -612,5 +612,5 @@
   </link>
   <!-- Joint from part_1 to part_36 -->
-  <joint name="rearwheel" type="revolute">
+  <joint name="rear_wheel_joint" type="revolute">
     <origin xyz="-0.0623407 -0.0348985 0.0485928" rpy="-1.5708 0.506098 1.5708"/>
     <parent link="part_1"/>
@@ -644,5 +644,5 @@
   </link>
   <!-- Joint from part_1 to part_35 -->
-  <joint name="leftwheel" type="revolute">
+  <joint name="left_wheel_joint" type="revolute">
     <origin xyz="-0.245137 0.278747 0.14524" rpy="-1.5708 -0 -1.5708"/>
     <parent link="part_1"/>
@@ -676,5 +676,5 @@
   </link>
   <!-- Joint from part_1 to part_34 -->
-  <joint name="rightwheel" type="revolute">
+  <joint name="right_wheel_joint" type="revolute">
     <origin xyz="0.171423 0.278747 0.14524" rpy="-1.5708 -0 1.5708"/>
     <parent link="part_1"/>
@@ -708,5 +708,5 @@
   </link>
   <!-- Joint from part_1 to part_37 -->
-  <joint name="frontwheel" type="revolute">
+  <joint name="front_wheel_joint" type="revolute">
     <origin xyz="-0.0622571 0.659747 0.0658648" rpy="-1.5708 -0 1.5708"/>
     <parent link="part_1"/>

Commit message: proper straight driving

File: src/igvc_description/urdf/model.urdf.xacro (robot description, xacro)
@@ -612,5 +612,5 @@
   </link>
   <!-- Joint from part_1 to part_36 -->
-  <joint name="rear_wheel_joint" type="revolute">
+  <joint name="rear_wheel_joint" type="continuous">
     <origin xyz="-0.0623407 -0.0348985 0.0485928" rpy="-1.5708 0.506098 1.5708"/>
     <parent link="part_1"/>
@@ -644,9 +644,9 @@
   </link>
   <!-- Joint from part_1 to part_35 -->
-  <joint name="left_wheel_joint" type="revolute">
+  <joint name="left_wheel_joint" type="continuous">
     <origin xyz="-0.245137 0.278747 0.14524" rpy="-1.5708 -0 -1.5708"/>
     <parent link="part_1"/>
     <child link="part_35"/>
-    <axis xyz="0 0 1"/>
+    <axis xyz="0 0 -1"/>
     <limit effort="10" velocity="10" lower="-3.141592653589793" upper="3.141592653589793"/>
   </joint>
@@ -676,5 +676,5 @@
   </link>
   <!-- Joint from part_1 to part_34 -->
-  <joint name="right_wheel_joint" type="revolute">
+  <joint name="right_wheel_joint" type="continuous">
     <origin xyz="0.171423 0.278747 0.14524" rpy="-1.5708 -0 1.5708"/>
     <parent link="part_1"/>
@@ -708,5 +708,5 @@
   </link>
   <!-- Joint from part_1 to part_37 -->
-  <joint name="front_wheel_joint" type="revolute">
+  <joint name="front_wheel_joint" type="continuous">
     <origin xyz="-0.0622571 0.659747 0.0658648" rpy="-1.5708 -0 1.5708"/>
     <parent link="part_1"/>
