Commit message: Add whole-project bringup files (#21)
* Transition Hardware package to igvc_hardware

* Create nav, gazebo, slam packages

* Create description package

* Modify igvc_description CMakeLists

* Add oak description to decription package

* Remove placeholder uml

* implement navigation package

* Implement slam package, TODO tune for igvc

* Remove redundant CMake library targets

* Generate low fidelity sim model URDF

* Add onshape-to-robot config file

* Rename otr urdf to model

* Create robot urdf file

* Add rviz launch files

* Change hardware package name to igvc_hardware

* Correct project name in slam package cmakelist

* Correct meshes to assets in description cmake

* Remove references to deprecated urdf file

* add package name to URDF meshes (automate this in the future)

* Remove nonexistent adi rosdep

* Remove nonexistent odrive rosdep

* Add gz and gz control plugin to gazebo dependencies

* Add directories to gazebo cmake

* Implement empty world files

* Rename robot in launch file

* Placeholder sensor simulation and bridge configuration

* Add config directory to gazebo cmake

* Split rviz and publisher into separate launches

* Include publisher launch file in gazebo launch

* Remove unused imports

* Configure RGBD camera description

* Remove madgwick filter from sim launch file

* rename launch file to hardware.launch.py

* Update hardware bringups to have the proper ODrive drivetrain

* Add IMU node to hardware launch

* rename hardware xacro

* Add hardware xacro to robot xacro

* remove joint state broadcaster from controllers yaml

* Update src/igvc_gazebo/launch/empty_world.launch.py

Co-authored-by: Mathew Davis <mjdavis0504@gmail.com>

* Update src/igvc_gazebo/launch/empty_world.launch.py

Co-authored-by: Mathew Davis <mjdavis0504@gmail.com>

* Fix file URDF locations

* Reconfigure robot description to use hardware package for ros2 control

* Remove duplicate OAK and position existing camera

* Change oak name, add igvc_robot to sensor xacro

* Fix devcontainer symlink install

* add friction to ground plane

* Change sensor formatting to recommended format

* Update bridge topic names

* Alter inertial values

* Change robot spawn location

* Reconfigure OAK simulation URDF

* Change rtabmap sim launch

* Add igvc_bringup

* Add control.launch.py

* Remove some extraneous elements and add CMakeLists

* Refactor bringup references

* Small refactor to hardware bringups

* Fix path substitution

* Working selection of sim scenario

* Almost running, controller manager dying on launch

* oops don't need that

* comment extraenous stuff

* Pass use_mock_hardware through publisher launch

* Add type to bot_drive_controller

* Add config to cmakelist

* add state interfaces to wheel joints

* Ros2 control actually runs! It was an error in rclcpp

* remove publisher node from empty world launch file

* Remove unused launch file

* remove nav2 bringup from launch file

* Update launch configuration names for clarity

* Move bot.ros2_control.xacro to igvc_description

* fix some config issues

---------

Co-authored-by: Zane Brotherton <zanebrotherton@gmail.com>
Co-authored-by: Zane Brotherton <46907447+zbrotherton@users.noreply.github.com>
Co-authored-by: Mathew Davis <mjdavis0504@gmail.com>
Co-authored-by: Spilsed <93678295+Spilsed@users.noreply.github.com>

File: src/igvc_description/urdf/model.urdf.xacro (robot description, xacro)
@@ -644,5 +644,5 @@
   </link>
   <!-- Joint from part_1 to part_35 -->
-  <joint name="leftwheel" type="revolute">
+  <joint name="left_wheel_joint" type="revolute">
     <origin xyz="-0.245137 0.278747 0.14524" rpy="-1.5708 -0 -1.5708"/>
     <parent link="part_1"/>
@@ -676,5 +676,5 @@
   </link>
   <!-- Joint from part_1 to part_34 -->
-  <joint name="rightwheel" type="revolute">
+  <joint name="right_wheel_joint" type="revolute">
     <origin xyz="0.171423 0.278747 0.14524" rpy="-1.5708 -0 1.5708"/>
     <parent link="part_1"/>
