Commit message: Added new model, does not load into sim yet

File: src/igvc_description/urdf/model.urdf.xacro (robot description, xacro)
@@ -1,8 +1,8 @@
 <?xml version="1.0" ?>
 <!-- Generated using onshape-to-robot -->
-<!-- Onshape https://cad.onshape.com/documents/4f27315f66a4121bf8434c1a/w/bce24b18b959f9c2227327f4/e/534f540c791514c4a2b9f32e -->
+<!-- Onshape https://cad.onshape.com/documents/e6f73c86a08716a88fa88928/w/70364c3c27402afccfdf9175/e/f88ba1396c902cb40ba93f4c -->
 <robot name="igvc_description">
-  <!-- Link part_1 -->
-  <link name="part_1">
+  <!-- Link igvc26_001 -->
+  <link name="igvc26_001">
     <inertial>
       <origin xyz="-0.0368571 0.291615 0.214315" rpy="0 0 0"/>
@@ -10,103 +10,23 @@
       <inertia ixx="3.60749" ixy="0" ixz="0" iyy="1.28472" iyz="0.159952" izz="3.84124"/>
     </inertial>
-    <!-- Part part_9 -->
-    <visual>
-      <origin xyz="-0.0368571 -0.178453 0.142065" rpy="0 -0 0"/>
-      <geometry>
-        <mesh filename="file://$(find igvc_description)/assets/part_9.stl"/>
-      </geometry>
-      <material name="part_9_material">
-        <color rgba="0.647059 0.647059 0.647059 1"/>
-      </material>
-    </visual>
-    <collision>
-      <origin xyz="-0.0368571 -0.178453 0.142065" rpy="0 -0 0"/>
-      <geometry>
-        <mesh filename="file://$(find igvc_description)/assets/part_9.stl"/>
-      </geometry>
-    </collision>
-    <!-- Part part_33 -->
-    <visual>
-      <origin xyz="-0.0368571 -0.178453 0.142065" rpy="0 -0 0"/>
-      <geometry>
-        <mesh filename="file://$(find igvc_description)/assets/part_33.stl"/>
-      </geometry>
-      <material name="part_33_material">
-        <color rgba="1 0 0 1"/>
-      </material>
-    </visual>
-    <collision>
-      <origin xyz="-0.0368571 -0.178453 0.142065" rpy="0 -0 0"/>
-      <geometry>
-        <mesh filename="file://$(find igvc_description)/assets/part_33.stl"/>
-      </geometry>
-    </collision>
-    <!-- Part part_14 -->
-    <visual>
-      <origin xyz="-0.0368571 -0.178453 0.142065" rpy="0 -0 0"/>
-      <geometry>
-        <mesh filename="file://$(find igvc_description)/assets/part_14.stl"/>
-      </geometry>
-      <material name="part_14_material">
-        <color rgba="0.647059 0.647059 0.647059 1"/>
-      </material>
-    </visual>
-    <collision>
-      <origin xyz="-0.0368571 -0.178453 0.142065" rpy="0 -0 0"/>
-      <geometry>
-        <mesh filename="file://$(find igvc_description)/assets/part_14.stl"/>
-      </geometry>
-    </collision>
-    <!-- Part part_23 -->
-    <visual>
-      <origin xyz="-0.0368571 -0.178453 0.142065" rpy="0 -0 0"/>
-      <geometry>
-        <mesh filename="file://$(find igvc_description)/assets/part_23.stl"/>
-      </geometry>
-      <material name="part_23_material">
-        <color rgba="0.647059 0.647059 0.647059 1"/>
-      </material>
-    </visual>
-    <collision>
-      <origin xyz="-0.0368571 -0.178453 0.142065" rpy="0 -0 0"/>
-      <geometry>
-        <mesh filename="file://$(find igvc_description)/assets/part_23.stl"/>
-      </geometry>
-    </collision>
-    <!-- Part part_5 -->
-    <visual>
-      <origin xyz="-0.0368571 -0.178453 0.142065" rpy="0 -0 0"/>
-      <geometry>
-        <mesh filename="file://$(find igvc_description)/assets/part_5.stl"/>
-      </geometry>
-      <material name="part_5_material">
-        <color rgba="0.647059 0.647059 0.647059 1"/>
-      </material>
-    </visual>
-    <collision>
-      <origin xyz="-0.0368571 -0.178453 0.142065" rpy="0 -0 0"/>
-      <geometry>
-        <mesh filename="file://$(find igvc_description)/assets/part_5.stl"/>
-      </geometry>
-    </collision>
-    <!-- Part part_1 -->
-    <visual>
-      <origin xyz="-0.0368571 -0.178453 0.142065" rpy="0 -0 0"/>
-      <geometry>
-        <mesh filename="file://$(find igvc_description)/assets/part_1.stl"/>
-      </geometry>
-      <material name="part_1_material">
-        <color rgba="0.647059 0.647059 0.647059 1"/>
-      </material>
-    </visual>
-    <collision>
-      <origin xyz="-0.0368571 -0.178453 0.142065" rpy="0 -0 0"/>
-      <geometry>
-        <mesh filename="file://$(find igvc_description)/assets/part_1.stl"/>
+    <!-- Part t_gusset__sharp_corners___10__0_098__thick___configuration_t_gusset__sharp_corners -->
+    <visual>
+      <origin xyz="0.416445 0.113415 -0.0766893" rpy="-1.5708 -4.0431e-08 1.06926"/>
+      <geometry>
+        <mesh filename="file://$(find igvc_description)/assets/t_gusset__sharp_corners___10__0_098__thick___configuration_t_gusset__sharp_corners.stl"/>
+      </geometry>
+      <material name="t_gusset__sharp_corners___10__0_098__thick___configuration_t_gusset__sharp_corners_material">
+        <color rgba="0.901961 0.901961 0.901961 1"/>
+      </material>
+    </visual>
+    <collision>
+      <origin xyz="0.416445 0.113415 -0.0766893" rpy="-1.5708 -4.0431e-08 1.06926"/>
+      <geometry>
+        <mesh filename="file://$(find igvc_description)/assets/t_gusset__sharp_corners___10__0_098__thick___configuration_t_gusset__sharp_corners.stl"/>
       </geometry>
     </collision>
     <!-- Part part_28 -->
     <visual>
-      <origin xyz="-0.0368571 -0.178453 0.142065" rpy="0 -0 0"/>
+      <origin xyz="0.39351 0.212892 -0.0500392" rpy="1.6076e-08 -4.0431e-08 1.06926"/>
       <geometry>
         <mesh filename="file://$(find igvc_description)/assets/part_28.stl"/>
@@ -117,476 +37,1116 @@
     </visual>
     <collision>
-      <origin xyz="-0.0368571 -0.178453 0.142065" rpy="0 -0 0"/>
+      <origin xyz="0.39351 0.212892 -0.0500392" rpy="1.6076e-08 -4.0431e-08 1.06926"/>
       <geometry>
         <mesh filename="file://$(find igvc_description)/assets/part_28.stl"/>
       </geometry>
     </collision>
-    <!-- Part part_12 -->
-    <visual>
-      <origin xyz="-0.0368571 -0.178453 0.142065" rpy="0 -0 0"/>
-      <geometry>
-        <mesh filename="file://$(find igvc_description)/assets/part_12.stl"/>
-      </geometry>
-      <material name="part_12_material">
-        <color rgba="0.647059 0.647059 0.647059 1"/>
-      </material>
-    </visual>
-    <collision>
-      <origin xyz="-0.0368571 -0.178453 0.142065" rpy="0 -0 0"/>
-      <geometry>
-        <mesh filename="file://$(find igvc_description)/assets/part_12.stl"/>
-      </geometry>
-    </collision>
-    <!-- Part part_30 -->
-    <visual>
-      <origin xyz="-0.0368571 -0.178453 0.142065" rpy="0 -0 0"/>
-      <geometry>
-        <mesh filename="file://$(find igvc_description)/assets/part_30.stl"/>
-      </geometry>
-      <material name="part_30_material">
+    <!-- Part igvc26_022 -->
+    <visual>
+      <origin xyz="0.0538636 0.399118 0.0515608" rpy="1.6076e-08 -4.0431e-08 1.06926"/>
+      <geometry>
+        <mesh filename="file://$(find igvc_description)/assets/igvc26_022.stl"/>
+      </geometry>
+      <material name="igvc26_022_material">
+        <color rgba="0.615686 0.811765 0.929412 0.498039"/>
+      </material>
+    </visual>
+    <collision>
+      <origin xyz="0.0538636 0.399118 0.0515608" rpy="1.6076e-08 -4.0431e-08 1.06926"/>
+      <geometry>
+        <mesh filename="file://$(find igvc_description)/assets/igvc26_022.stl"/>
+      </geometry>
+    </collision>
+    <!-- Part wcp_2103_rev2 -->
+    <visual>
+      <origin xyz="0.190503 0.546513 -0.0214642" rpy="-1.5708 1.45917 2.64006"/>
+      <geometry>
+        <mesh filename="file://$(find igvc_description)/assets/wcp_2103_rev2.stl"/>
+      </geometry>
+      <material name="wcp_2103_rev2_material">
+        <color rgba="0.792157 0.819608 0.933333 1"/>
+      </material>
+    </visual>
+    <collision>
+      <origin xyz="0.190503 0.546513 -0.0214642" rpy="-1.5708 1.45917 2.64006"/>
+      <geometry>
+        <mesh filename="file://$(find igvc_description)/assets/wcp_2103_rev2.stl"/>
+      </geometry>
+    </collision>
+    <!-- Part igvc26_013 -->
+    <visual>
+      <origin xyz="0.139416 0.462431 -0.0563892" rpy="1.6076e-08 -4.0431e-08 1.06926"/>
+      <geometry>
+        <mesh filename="file://$(find igvc_description)/assets/igvc26_013.stl"/>
+      </geometry>
+      <material name="igvc26_013_material">
+        <color rgba="0.917647 0.917647 0.917647 1"/>
+      </material>
+    </visual>
+    <collision>
+      <origin xyz="0.139416 0.462431 -0.0563892" rpy="1.6076e-08 -4.0431e-08 1.06926"/>
+      <geometry>
+        <mesh filename="file://$(find igvc_description)/assets/igvc26_013.stl"/>
+      </geometry>
+    </collision>
+    <!-- Part igvc26_003 -->
+    <visual>
+      <origin xyz="-0.171736 1.1724 -0.0627392" rpy="-4.0431e-08 -1.6076e-08 2.64006"/>
+      <geometry>
+        <mesh filename="file://$(find igvc_description)/assets/igvc26_003.stl"/>
+      </geometry>
+      <material name="igvc26_003_material">
+        <color rgba="0.647059 0.647059 0.647059 1"/>
+      </material>
+    </visual>
+    <collision>
+      <origin xyz="-0.171736 1.1724 -0.0627392" rpy="-4.0431e-08 -1.6076e-08 2.64006"/>
+      <geometry>
+        <mesh filename="file://$(find igvc_description)/assets/igvc26_003.stl"/>
+      </geometry>
+    </collision>
+    <!-- Part igvc26_023 -->
+    <visual>
+      <origin xyz="-0.362056 0.627164 -0.0754392" rpy="1.6076e-08 -4.0431e-08 1.06926"/>
+      <geometry>
+        <mesh filename="file://$(find igvc_description)/assets/igvc26_023.stl"/>
+      </geometry>
+      <material name="igvc26_023_material">
+        <color rgba="0.25098 0.482353 0.992157 0.2"/>
+      </material>
+    </visual>
+    <collision>
+      <origin xyz="-0.362056 0.627164 -0.0754392" rpy="1.6076e-08 -4.0431e-08 1.06926"/>
+      <geometry>
+        <mesh filename="file://$(find igvc_description)/assets/igvc26_023.stl"/>
+      </geometry>
+    </collision>
+    <!-- Part igvc26_011 -->
+    <visual>
+      <origin xyz="0.0538636 0.399118 -0.0500392" rpy="1.6076e-08 -4.0431e-08 1.06926"/>
+      <geometry>
+        <mesh filename="file://$(find igvc_description)/assets/igvc26_011.stl"/>
+      </geometry>
+      <material name="igvc26_011_material">
+        <color rgba="0.615686 0.811765 0.929412 0.498039"/>
+      </material>
+    </visual>
+    <collision>
+      <origin xyz="0.0538636 0.399118 -0.0500392" rpy="1.6076e-08 -4.0431e-08 1.06926"/>
+      <geometry>
+        <mesh filename="file://$(find igvc_description)/assets/igvc26_011.stl"/>
+      </geometry>
+    </collision>
+    <!-- Part igvc26_013_2 -->
+    <visual>
+      <origin xyz="0.0612413 0.505294 -0.0563892" rpy="1.6076e-08 -4.0431e-08 1.06926"/>
+      <geometry>
+        <mesh filename="file://$(find igvc_description)/assets/igvc26_013.stl"/>
+      </geometry>
+      <material name="igvc26_013_2_material">
+        <color rgba="0.917647 0.917647 0.917647 1"/>
+      </material>
+    </visual>
+    <collision>
+      <origin xyz="0.0612413 0.505294 -0.0563892" rpy="1.6076e-08 -4.0431e-08 1.06926"/>
+      <geometry>
+        <mesh filename="file://$(find igvc_description)/assets/igvc26_013.stl"/>
+      </geometry>
+    </collision>
+    <!-- Part igvc26_015 -->
+    <visual>
+      <origin xyz="0.0267798 0.728242 -0.0563892" rpy="1.6076e-08 -4.0431e-08 1.06926"/>
+      <geometry>
+        <mesh filename="file://$(find igvc_description)/assets/igvc26_015.stl"/>
+      </geometry>
+      <material name="igvc26_015_material">
+        <color rgba="0.972549 0.529412 0.00392157 1"/>
+      </material>
+    </visual>
+    <collision>
+      <origin xyz="0.0267798 0.728242 -0.0563892" rpy="1.6076e-08 -4.0431e-08 1.06926"/>
+      <geometry>
+        <mesh filename="file://$(find igvc_description)/assets/igvc26_015.stl"/>
+      </geometry>
+    </collision>
+    <!-- Part igvc26_006 -->
+    <visual>
+      <origin xyz="0.2153 0.482224 -0.0627392" rpy="-1.6076e-08 4.0431e-08 -2.07233"/>
+      <geometry>
+        <mesh filename="file://$(find igvc_description)/assets/igvc26_006.stl"/>
+      </geometry>
+      <material name="igvc26_006_material">
+        <color rgba="0.972549 0.529412 0.00392157 1"/>
+      </material>
+    </visual>
+    <collision>
+      <origin xyz="0.2153 0.482224 -0.0627392" rpy="-1.6076e-08 4.0431e-08 -2.07233"/>
+      <geometry>
+        <mesh filename="file://$(find igvc_description)/assets/igvc26_006.stl"/>
+      </geometry>
+    </collision>
+    <!-- Part igvc26_015_2 -->
+    <visual>
+      <origin xyz="-0.306153 0.596513 -0.0563892" rpy="1.6076e-08 -4.0431e-08 1.06926"/>
+      <geometry>
+        <mesh filename="file://$(find igvc_description)/assets/igvc26_015.stl"/>
+      </geometry>
+      <material name="igvc26_015_2_material">
+        <color rgba="0.972549 0.529412 0.00392157 1"/>
+      </material>
+    </visual>
+    <collision>
+      <origin xyz="-0.306153 0.596513 -0.0563892" rpy="1.6076e-08 -4.0431e-08 1.06926"/>
+      <geometry>
+        <mesh filename="file://$(find igvc_description)/assets/igvc26_015.stl"/>
+      </geometry>
+    </collision>
+    <!-- Part wcp_2103_rev2_2 -->
+    <visual>
+      <origin xyz="0.00631191 0.202876 -0.0214643" rpy="2.07233 1.5708 0"/>
+      <geometry>
+        <mesh filename="file://$(find igvc_description)/assets/wcp_2103_rev2.stl"/>
+      </geometry>
+      <material name="wcp_2103_rev2_2_material">
+        <color rgba="0.792157 0.819608 0.933333 1"/>
+      </material>
+    </visual>
+    <collision>
+      <origin xyz="0.00631191 0.202876 -0.0214643" rpy="2.07233 1.5708 0"/>
+      <geometry>
+        <mesh filename="file://$(find igvc_description)/assets/wcp_2103_rev2.stl"/>
+      </geometry>
+    </collision>
+    <!-- Part right_triangle_gusset -->
+    <visual>
+      <origin xyz="-0.362517 0.613187 -0.0414198" rpy="1.6076e-08 -4.0431e-08 1.06926"/>
+      <geometry>
+        <mesh filename="file://$(find igvc_description)/assets/right_triangle_gusset.stl"/>
+      </geometry>
+      <material name="right_triangle_gusset_material">
+        <color rgba="0.282353 0.54902 0.160784 1"/>
+      </material>
+    </visual>
+    <collision>
+      <origin xyz="-0.362517 0.613187 -0.0414198" rpy="1.6076e-08 -4.0431e-08 1.06926"/>
+      <geometry>
+        <mesh filename="file://$(find igvc_description)/assets/right_triangle_gusset.stl"/>
+      </geometry>
+    </collision>
+    <!-- Part left_triangle_gusset -->
+    <visual>
+      <origin xyz="-0.362594 0.612975 -0.0436892" rpy="1.6076e-08 -4.0431e-08 1.06926"/>
+      <geometry>
+        <mesh filename="file://$(find igvc_description)/assets/left_triangle_gusset.stl"/>
+      </geometry>
+      <material name="left_triangle_gusset_material">
+        <color rgba="0.282353 0.54902 0.160784 1"/>
+      </material>
+    </visual>
+    <collision>
+      <origin xyz="-0.362594 0.612975 -0.0436892" rpy="1.6076e-08 -4.0431e-08 1.06926"/>
+      <geometry>
+        <mesh filename="file://$(find igvc_description)/assets/left_triangle_gusset.stl"/>
+      </geometry>
+    </collision>
+    <!-- Part igvc26_019 -->
+    <visual>
+      <origin xyz="0.0538636 0.399118 -0.0627392" rpy="1.6076e-08 -4.0431e-08 1.06926"/>
+      <geometry>
+        <mesh filename="file://$(find igvc_description)/assets/igvc26_019.stl"/>
+      </geometry>
+      <material name="igvc26_019_material">
+        <color rgba="0.615686 0.811765 0.929412 0.498039"/>
+      </material>
+    </visual>
+    <collision>
+      <origin xyz="0.0538636 0.399118 -0.0627392" rpy="1.6076e-08 -4.0431e-08 1.06926"/>
+      <geometry>
+        <mesh filename="file://$(find igvc_description)/assets/igvc26_019.stl"/>
+      </geometry>
+    </collision>
+    <!-- Part 135_degree_gusset___10__0_098__thick___configuration__135_degree -->
+    <visual>
+      <origin xyz="-0.32561 0.261755 -0.0766892" rpy="1.5708 -3.9956e-08 1.85466"/>
+      <geometry>
+        <mesh filename="file://$(find igvc_description)/assets/135_degree_gusset___10__0_098__thick___configuration__135_degree.stl"/>
+      </geometry>
+      <material name="135_degree_gusset___10__0_098__thick___configuration__135_degree_material">
+        <color rgba="0.901961 0.901961 0.901961 1"/>
+      </material>
+    </visual>
+    <collision>
+      <origin xyz="-0.32561 0.261755 -0.0766892" rpy="1.5708 -3.9956e-08 1.85466"/>
+      <geometry>
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
File: src/igvc_description/urdf/sensor/camera.urdf.xacro (robot description, xacro)
@@ -1,72 +1,112 @@
-<?xml version="1.0" ?>
+<?xml version="1.0"?>
 <robot xmlns:xacro="http://www.ros.org/wiki/xacro">
-    <xacro:arg name="camera_name"   default="oak" />
-    <xacro:arg name="camera_model"  default="OAK-D-POE" />
-    <xacro:arg name="base_frame"    default="oak_base" />
-    <xacro:arg name="parent_frame"  default="oak_parent" />
-    <xacro:arg name="cam_pos_x"     default="0.0" />
-    <xacro:arg name="cam_pos_y"     default="0.0" />
-    <xacro:arg name="cam_pos_z"     default="0.0" />
-    <xacro:arg name="cam_roll"      default="0.0" />
-    <xacro:arg name="cam_pitch"     default="0.0" />
-    <xacro:arg name="cam_yaw"       default="0.0" />
-    <xacro:arg name="rs_compat"     default="true" />
-    <xacro:include filename="$(find depthai_descriptions)/urdf/depthai_descr.urdf.xacro" />
-    <joint name="camera_base_joint" type="fixed">
-        <parent link="base_footprint"/>
-        <child link="oak_parent"/>
-        <origin xyz="-0.05 -0.05 0.95" rpy="0 0 ${pi/2}"/>
-    </joint>
-    <gazebo reference="oak_color_frame">
-        <sensor name="oak_depth" type="depth">
-            <pose> 0 0 0 0 0 0 </pose>
-            <topic>oak/depth</topic>
-            <update_rate>20</update_rate>
-            <always_on>1</always_on>
-            <gz_frame_id>oak_color_optical_frame</gz_frame_id>
-            <camera>
-                <horizontal_fov>1.51843645</horizontal_fov>
-                <image>
-                    <format>R_FLOAT32</format>
-                    <width>1280</width>
-                    <height>720</height>
-                </image>
-                <clip>
-                    <near>0.28</near>
-                    <far>10</far>
-                </clip>
-            </camera>
-            <plugin filename="libgz-sim8-sensors-system.so" name="gz::sim::v8::systems::Sensors"></plugin>
-        </sensor>
-    </gazebo>
-    <gazebo reference="oak_color_frame">
-        <sensor name="camera" type="camera">
-            <camera>
-                <horizontal_fov>1.51843645</horizontal_fov>
-                <image>
-                    <width>1280</width>
-                    <height>720</height>
-                    <format>R8G8B8</format>
-                </image>
-                <clip>
-                    <near>0.05</near>
-                    <far>20</far>
-                </clip>
-                <noise>
-                    <type>gaussian</type>
-                    <!-- Noise is sampled independently per pixel on each frame.
-                        That pixel's noise value is added to each of its color
-                        channels, which at that point lie in the range [0,1]. -->
-                    <mean>0.0</mean>
-                    <stddev>0.007</stddev>
-                </noise>
-                <optical_frame_id>oak_color_optical_frame</optical_frame_id>
-                <camera_info_topic>oak/camera_info</camera_info_topic>
-            </camera>
-            <always_on>1</always_on>
-            <update_rate>20</update_rate>
-            <visualize>true</visualize>
-            <topic>oak/color</topic>
-        </sensor>
-    </gazebo>
+  <link name="zed2i_base_link">
+    <visual>
+      <geometry>
+        <box size="0.175 0.03 0.03"/>
+      </geometry>
+      <material name="black"/>
+    </visual>
+  </link>
+  <joint name="camera_base_joint" type="fixed">
+    <parent link="base_footprint"/>
+    <child link="zed2i_base_link"/>
+    <origin xyz="-0.05 -0.05 0.95" rpy="0 0 1.5708"/>
+  </joint>
+  <link name="zed2i_left_camera_frame"/>
+  <joint name="zed2i_left_joint" type="fixed">
+    <parent link="zed2i_base_link"/>
+    <child link="zed2i_left_camera_frame"/>
+    <origin xyz="0 0.03 0" rpy="0 0 0"/>
+  </joint>
+  <link name="zed2i_left_camera_optical_frame"/>
+  <joint name="zed2i_left_optical_joint" type="fixed">
+    <parent link="zed2i_left_camera_frame"/>
+    <child link="zed2i_left_camera_optical_frame"/>
+    <origin xyz="0 0 0" rpy="-1.5708 0 -1.5708"/>
+  </joint>
+  <link name="zed2i_right_camera_frame"/>
+  <joint name="zed2i_right_joint" type="fixed">
+    <parent link="zed2i_base_link"/>
+    <child link="zed2i_right_camera_frame"/>
+    <origin xyz="0 -0.03 0" rpy="0 0 0"/>
+  </joint>
+  <link name="zed2i_right_camera_optical_frame"/>
+  <joint name="zed2i_right_optical_joint" type="fixed">
+    <parent link="zed2i_right_camera_frame"/>
+    <child link="zed2i_right_camera_optical_frame"/>
+    <origin xyz="0 0 0" rpy="-1.5708 0 -1.5708"/>
+  </joint>
+  <gazebo reference="zed2i_left_camera_frame">
+    <sensor name="zed2i_rgb" type="camera">
+      <pose>0 0 0 0 0 0</pose>
+      <camera>
+        <horizontal_fov>1.5708</horizontal_fov>
+        <image>
+          <width>1280</width>
+          <height>720</height>
+          <format>R8G8B8</format>
+        </image>
+        <clip>
+          <near>0.05</near>
+          <far>30.0</far>
+        </clip>
+        <noise>
+          <type>gaussian</type>
+          <mean>0.0</mean>
+          <stddev>0.005</stddev>
+        </noise>
+        <optical_frame_id>zed2i_left_camera_optical_frame</optical_frame_id>
+        <camera_info_topic>zed2i/camera_info</camera_info_topic>
+      </camera>
+      <always_on>1</always_on>
+      <update_rate>30</update_rate>
+      <visualize>true</visualize>
+      <topic>zed2i/image_raw</topic>
+    </sensor>
+  </gazebo>
+  <gazebo reference="zed2i_left_camera_frame">
+    <sensor name="zed2i_depth" type="depth">
+      <pose>0 0 0 0 0 0</pose>
+      <topic>zed2i/depth</topic>
+      <update_rate>30</update_rate>
+      <always_on>1</always_on>
+      <gz_frame_id>zed2i_left_camera_optical_frame</gz_frame_id>
+      <camera>
+        <horizontal_fov>1.5708</horizontal_fov>
+        <image>
+          <width>1280</width>
+          <height>720</height>
+          <format>R_FLOAT32</format>
+        </image>
+        <clip>
+          <near>0.3</near>
+          <far>20.0</far>
+        </clip>
+      </camera>
+      <plugin filename="libgz-sim8-sensors-system.so"
+              name="gz::sim::v8::systems::Sensors"/>
+    </sensor>
+  </gazebo>
+  <gazebo reference="zed2i_right_camera_frame">
+    <sensor name="zed2i_right" type="camera">
+      <pose>0 0 0 0 0 0</pose>
+      <camera>
+        <horizontal_fov>1.5708</horizontal_fov>
+        <image>
+          <width>1280</width>
+          <height>720</height>
+          <format>R8G8B8</format>
+        </image>
+        <clip>
+          <near>0.05</near>
+          <far>30.0</far>
+        </clip>
+        <optical_frame_id>zed2i_right_camera_optical_frame</optical_frame_id>
+      </camera>
+      <always_on>1</always_on>
+      <update_rate>30</update_rate>
+      <topic>zed2i/right/image_raw</topic>
+    </sensor>
+  </gazebo>
 </robot>
