Commit message: Create robot urdf file

File: src/igvc_description/urdf/robot.urdf.xacro (robot description, xacro)
@@ -1,16 +1,6 @@
 <?xml version="1.0" ?>
-<robot xmlns:xacro="http://www.ros.org/wiki/xacro" name="igvc_robot">
-    <xacro:arg name="prefix" default="" />
-    <xacro:arg name="use_mock_hardware" default="false" />
-    <link name="base_footprint"/>
-    <joint name="base_joint" type="fixed">
-        <parent link="base_footprint"/>
-        <origin rpy="0 0 0" xyz="0 0 0.15"/>
-        <child link="part_1"/>
-        <axis xyz="0 0 1"/>
-    </joint>
+<robot xmlns:xacro="http://www.ros.org/wiki/xacro" name="igvc">
     <xacro:include filename="$(find igvc_description)/urdf/model.urdf.xacro"/>
+    <xacro:include filename="$(find igvc_description)/urdf/control.urdf.xacro"/>
     <xacro:include filename="$(find igvc_description)/urdf/sensors.urdf.xacro"/>
-    <xacro:include filename="$(find igvc_hardware)/description/bot.ros2_control.xacro" />
-    <xacro:bot_ros2_control name="IGVC_Bot" prefix="$(arg prefix)" use_mock_hardware="$(arg use_mock_hardware)"/>
 </robot>

Commit message: Placeholder sensor simulation and bridge configuration

File: src/igvc_description/urdf/robot.urdf.xacro (robot description, xacro)
@@ -1,6 +1,13 @@
 <?xml version="1.0" ?>
-<robot xmlns:xacro="http://www.ros.org/wiki/xacro" name="igvc">
+<robot xmlns:xacro="http://www.ros.org/wiki/xacro" name="igvc_robot">
+    <link name="base_footprint"/>
+    <joint name="base_joint" type="fixed">
+        <parent link="base_footprint"/>
+        <origin rpy="0 0 0" xyz="0 0 0"/>
+        <child link="part_1"/>
+        <axis xyz="0 0 1"/>
+    </joint>
     <xacro:include filename="$(find igvc_description)/urdf/model.urdf.xacro"/>
-    <xacro:include filename="$(find igvc_description)/urdf/control.urdf.xacro"/>
-    <xacro:include filename="$(find igvc_description)/urdf/sensors.urdf.xacro"/>
+    <!-- <xacro:include filename="$(find igvc_description)/urdf/control.urdf.xacro"/> -->
+    <!-- <xacro:include filename="$(find igvc_description)/urdf/sensors.urdf.xacro"/> -->
 </robot>

Commit message: Configure RGBD camera description

File: src/igvc_description/urdf/robot.urdf.xacro (robot description, xacro)
@@ -10,4 +10,4 @@
     <xacro:include filename="$(find igvc_description)/urdf/model.urdf.xacro"/>
     <!-- <xacro:include filename="$(find igvc_description)/urdf/control.urdf.xacro"/> -->
-    <!-- <xacro:include filename="$(find igvc_description)/urdf/sensors.urdf.xacro"/> -->
+    <xacro:include filename="$(find igvc_description)/urdf/sensors.urdf.xacro"/>
 </robot>

File: src/igvc_description/urdf/sensors.urdf.xacro (robot description, xacro)
@@ -1,12 +1,27 @@
 <?xml version="1.0" ?>
 <robot xmlns:xacro="http://www.ros.org/wiki/xacro">
-    <xacro:include filename="$(find realsense2_description)/urdf/_d435i.urdf.xacro"/>
-    <xacro:sensor_d435i parent="base_link" use_nominal_extrinsics="false">
-        <origin xyz="0.169586 0.00312814 0.06" rpy="0 0 0"/>
-    </xacro:sensor_d435i>
-    <joint name="camera_optical_link" type="fixed">
+    <xacro:include filename="$(find depthai_descriptions)/urdf/depthai_descr.urdf.xacro"/>
+    <xacro:depthai_camera
+        camera_name="oak_depth"
+        camera_model="OAK-D-POE"
+        base_frame="camera_link"
+        parent="base_footprint"
+        cam_pos_x="0.0"
+        cam_pos_y="0.0"
+        cam_pos_z="0.0"
+        cam_roll="0.0"
+        cam_pitch="0.0"
+        cam_yaw="0.0"
+        rs_compat="true"
+    />
+    <joint name="camera_base_joint" type="fixed">
+        <parent link="base_footprint"/>
+        <child link="oak-d-base-frame"/>
         <origin xyz="0 0 0" rpy="${-pi/2} 0 ${-pi/2}"/>
+    </joint>
+    <joint name="camera_optical_joint" type="fixed">
         <parent link="camera_link"/>
         <child link="camera_link_optical"/>
+        <origin xyz="0 0 0" rpy="${-pi/2} 0 ${-pi/2}"/>
     </joint>
     <link name="camera_link_optical"></link>

Commit message: Change robot spawn location

File: src/igvc_description/urdf/robot.urdf.xacro (robot description, xacro)
@@ -6,5 +6,5 @@
     <joint name="base_joint" type="fixed">
         <parent link="base_footprint"/>
-        <origin rpy="0 0 0" xyz="0 0 0"/>
+        <origin rpy="0 0 0" xyz="0 0 0.15"/>
         <child link="part_1"/>
         <axis xyz="0 0 1"/>

Commit message: Create track world SDF (#88)
* Copy meshes into igvc_gazebo

* create track_v1 sdf

* change default in bringup to track v1

* Reposition robot and track locations

* Adjust sensor positions to be closer to real robot

* Add sky to simulation

* Remove ground plane, move track into ground plane

File: src/igvc_description/urdf/robot.urdf.xacro (robot description, xacro)
@@ -6,5 +6,5 @@
     <joint name="base_joint" type="fixed">
         <parent link="base_footprint"/>
-        <origin rpy="0 0 0" xyz="0 0 0.15"/>
+        <origin rpy="0 0 0" xyz="0 0 0.01"/>
         <child link="part_1"/>
         <axis xyz="0 0 1"/>

File: src/igvc_description/urdf/sensor/camera.urdf.xacro (robot description, xacro)
@@ -16,5 +16,5 @@
         <parent link="base_footprint"/>
         <child link="oak_parent"/>
-        <origin xyz="0 -0.4 0.95" rpy="0 0 ${pi/2}"/>
+        <origin xyz="-0.05 -0.05 0.95" rpy="0 0 ${pi/2}"/>
     </joint>
     <gazebo reference="oak_color_frame">

File: src/igvc_description/urdf/sensor/lidar.urdf.xacro (robot description, xacro)
@@ -4,5 +4,5 @@
         <parent link="base_footprint"/>
         <child link="laser_frame"/>
-        <origin xyz="0 0.2 0.50" rpy="0 0 0"/>
+        <origin xyz="-0.05 0.605 0.50" rpy="0 0 0"/>
     </joint>
     <link name="laser_frame">

Commit message: Draft of adding base_link

File: src/igvc_description/urdf/robot.urdf.xacro (robot description, xacro)
@@ -4,4 +4,11 @@
     <xacro:arg name="use_mock_hardware" default="false" />
     <link name="base_footprint"/>
+    <joint name="base_joint" type="fixed">
+        <parent link="base_footprint"/>
+        <origin rpy="0 0 0" xyz="0 0 0.01"/>
+        <child link="part_1"/>
+        <axis xyz="0 0 1"/>
+    </joint>
+    <link name="base_link"/>
     <joint name="base_joint" type="fixed">
         <parent link="base_footprint"/>

Commit message: Changed joint placement

File: src/igvc_description/urdf/robot.urdf.xacro (robot description, xacro)
@@ -4,13 +4,13 @@
     <xacro:arg name="use_mock_hardware" default="false" />
     <link name="base_footprint"/>
-    <joint name="base_joint" type="fixed">
-        <parent link="base_footprint"/>
+    <link name="base_link"/>
+    <joint name="footprint_joint" type="fixed">
+        <parent link="base_link"/>
         <origin rpy="0 0 0" xyz="0 0 0.01"/>
-        <child link="part_1"/>
+        <child link="base_footprint"/>
         <axis xyz="0 0 1"/>
     </joint>
-    <link name="base_link"/>
     <joint name="base_joint" type="fixed">
-        <parent link="base_footprint"/>
+        <parent link="base_link"/>
         <origin rpy="0 0 0" xyz="0 0 0.01"/>
         <child link="part_1"/>

Commit message: Moved base_footprint children to be children of base_link

File: src/igvc_description/urdf/robot.urdf.xacro (robot description, xacro)
@@ -5,4 +5,10 @@
     <link name="base_footprint"/>
     <link name="base_link"/>
+    <joint name="base_joint" type="fixed">
+        <parent link="base_link"/>
+        <origin rpy="0 0 0" xyz="0 0 0.01"/>
+        <child link="part_1"/>
+        <axis xyz="0 0 1"/>
+    </joint>
     <joint name="footprint_joint" type="fixed">
         <parent link="base_link"/>
@@ -11,8 +17,26 @@
         <axis xyz="0 0 1"/>
     </joint>
-    <joint name="base_joint" type="fixed">
+    <joint name="oak_joint" type="fixed">
         <parent link="base_link"/>
         <origin rpy="0 0 0" xyz="0 0 0.01"/>
-        <child link="part_1"/>
+        <child link="oak_parent"/>
+        <axis xyz="0 0 1"/>
+    </joint>
+    <joint name="imu_joint_link" type="fixed">
+        <parent link="base_link"/>
+        <origin rpy="0 0 0" xyz="0 0 0.01"/>
+        <child link="imu_link"/>
+        <axis xyz="0 0 1"/>
+    </joint>
+    <joint name="laser_joint_link" type="fixed">
+        <parent link="base_link"/>
+        <origin rpy="0 0 0" xyz="0 0 0.01"/>
+        <child link="laser_frame"/>
+        <axis xyz="0 0 1"/>
+    </joint>
+    <joint name="navsat_joint_link" type="fixed">
+        <parent link="base_link"/>
+        <origin rpy="0 0 0" xyz="0 0 0.01"/>
+        <child link="navsat_link"/>
         <axis xyz="0 0 1"/>
     </joint>

Commit message: Moved odom to be parent of base_link

File: src/igvc_description/urdf/robot.urdf.xacro (robot description, xacro)
@@ -5,4 +5,11 @@
     <link name="base_footprint"/>
     <link name="base_link"/>
+    <link name="odom"/>
+    <joint name="odom_joint" type="fixed">
+        <parent link="odom"/>
+        <origin rpy="0 0 0" xyz="0 0 0.01"/>
+        <child link="base_link"/>
+        <axis xyz="0 0 1"/>
+    </joint>
     <joint name="base_joint" type="fixed">
         <parent link="base_link"/>

Commit message: Changed sensor files instead of creating new joints

File: src/igvc_description/urdf/robot.urdf.xacro (robot description, xacro)
@@ -24,28 +24,4 @@
         <axis xyz="0 0 1"/>
     </joint>
-    <joint name="oak_joint" type="fixed">
-        <parent link="base_link"/>
-        <origin rpy="0 0 0" xyz="0 0 0.01"/>
-        <child link="oak_parent"/>
-        <axis xyz="0 0 1"/>
-    </joint>
-    <joint name="imu_joint_link" type="fixed">
-        <parent link="base_link"/>
-        <origin rpy="0 0 0" xyz="0 0 0.01"/>
-        <child link="imu_link"/>
-        <axis xyz="0 0 1"/>
-    </joint>
-    <joint name="laser_joint_link" type="fixed">
-        <parent link="base_link"/>
-        <origin rpy="0 0 0" xyz="0 0 0.01"/>
-        <child link="laser_frame"/>
-        <axis xyz="0 0 1"/>
-    </joint>
-    <joint name="navsat_joint_link" type="fixed">
-        <parent link="base_link"/>
-        <origin rpy="0 0 0" xyz="0 0 0.01"/>
-        <child link="navsat_link"/>
-        <axis xyz="0 0 1"/>
-    </joint>
     <xacro:include filename="$(find igvc_description)/urdf/model.urdf.xacro"/>
     <xacro:include filename="$(find igvc_description)/urdf/sensors.urdf.xacro"/>

File: src/igvc_description/urdf/sensor/camera.urdf.xacro (robot description, xacro)
@@ -14,5 +14,5 @@
     <xacro:include filename="$(find depthai_descriptions)/urdf/depthai_descr.urdf.xacro" />
     <joint name="camera_base_joint" type="fixed">
-        <parent link="base_footprint"/>
+        <parent link="base_link"/>
         <child link="oak_parent"/>
         <origin xyz="-0.05 -0.05 0.95" rpy="0 0 ${pi/2}"/>

File: src/igvc_description/urdf/sensor/gps.urdf.xacro (robot description, xacro)
@@ -3,5 +3,5 @@
     <joint name="navsat_joint" type="fixed">
         <origin xyz="0 0 0" rpy="0 0 0" />
-        <parent link="base_footprint"/>
+        <parent link="base_link"/>
         <child link="navsat_link" />
     </joint>

File: src/igvc_description/urdf/sensor/imu.urdf.xacro (robot description, xacro)
@@ -3,5 +3,5 @@
     <joint name="imu_joint" type="fixed">
         <origin xyz="0 0 0" rpy="0 0 0" />
-        <parent link="base_footprint"/>
+        <parent link="base_link"/>
         <child link="imu_link" />
         </joint>

File: src/igvc_description/urdf/sensor/lidar.urdf.xacro (robot description, xacro)
@@ -2,5 +2,5 @@
 <robot xmlns:xacro="http://www.ros.org/wiki/xacro">
     <joint name="laser_joint" type="fixed">
-        <parent link="base_footprint"/>
+        <parent link="base_link"/>
         <child link="laser_frame"/>
         <origin xyz="-0.05 0.605 0.50" rpy="0 0 0"/>

Commit message: Changed base_footprint to base_link in parameters

File: src/igvc_description/urdf/robot.urdf.xacro (robot description, xacro)
@@ -5,11 +5,4 @@
     <link name="base_footprint"/>
     <link name="base_link"/>
-    <link name="odom"/>
-    <joint name="odom_joint" type="fixed">
-        <parent link="odom"/>
-        <origin rpy="0 0 0" xyz="0 0 0.01"/>
-        <child link="base_link"/>
-        <axis xyz="0 0 1"/>
-    </joint>
     <joint name="base_joint" type="fixed">
         <parent link="base_link"/>

Commit message: Feature/base link urdf (#105)
* Drafted 2d_lidar for rtabmap

* merge conflicts

* Fixed typo and added RGBD/FromDepth parameters

* Removed ODOM and edited parameters

* Updating commit

* Drafted 2d_lidar for rtabmap

* merge conflicts

* Fixed typo and added RGBD/FromDepth parameters

* Removed ODOM and edited parameters

* Draft of adding base_link

* Edited joint

* Changed joint placement

* Moved base_footprint children to be children of base_link

* Moved odom to be parent of base_link

* Changed sensor files instead of creating new joints

* Reverted lidar changes

* Changed base_footprint to base_link in parameters

* Changed frame id from base_footprint to base_link and changed /odom topic to odom

File: src/igvc_description/urdf/robot.urdf.xacro (robot description, xacro)
@@ -4,8 +4,15 @@
     <xacro:arg name="use_mock_hardware" default="false" />
     <link name="base_footprint"/>
+    <link name="base_link"/>
     <joint name="base_joint" type="fixed">
-        <parent link="base_footprint"/>
+        <parent link="base_link"/>
         <origin rpy="0 0 0" xyz="0 0 0.01"/>
         <child link="part_1"/>
+        <axis xyz="0 0 1"/>
+    </joint>
+    <joint name="footprint_joint" type="fixed">
+        <parent link="base_link"/>
+        <origin rpy="0 0 0" xyz="0 0 0.01"/>
+        <child link="base_footprint"/>
         <axis xyz="0 0 1"/>
     </joint>

Commit message: reverse base_link

File: src/igvc_description/urdf/robot.urdf.xacro (robot description, xacro)
@@ -7,5 +7,5 @@
     <joint name="base_joint" type="fixed">
         <parent link="base_link"/>
-        <origin rpy="0 0 0" xyz="0 0 0.01"/>
+        <origin rpy="0 0 ${pi}" xyz="0 0 0.01"/>
         <child link="part_1"/>
         <axis xyz="0 0 1"/>

Commit message: track testing changes

File: src/igvc_description/urdf/robot.urdf.xacro (robot description, xacro)
@@ -7,5 +7,5 @@
     <joint name="base_joint" type="fixed">
         <parent link="base_link"/>
-        <origin rpy="0 0 ${pi}" xyz="0 0 0.01"/>
+        <origin rpy="0 0 3.14159" xyz="0 0 0.01"/>
         <child link="part_1"/>
         <axis xyz="0 0 1"/>

Commit message: Checkpoint: Hail Mary

File: src/igvc_description/urdf/robot.urdf.xacro (robot description, xacro)
@@ -7,5 +7,5 @@
     <joint name="base_joint" type="fixed">
         <parent link="base_link"/>
-        <origin rpy="0 0 3.14159" xyz="0 0 0.01"/>
+        <origin rpy="0 0 0" xyz="0 0 0.01"/>
         <child link="part_1"/>
         <axis xyz="0 0 1"/>
