Commit message: remove oak from camera.urdf.xacro

File: src/igvc_description/urdf/sensor/camera.urdf.xacro (robot description, xacro)
@@ -1,19 +1,7 @@
 <?xml version="1.0" ?>
 <robot xmlns:xacro="http://www.ros.org/wiki/xacro">
-    <xacro:arg name="camera_name"   default="oak" />
-    <xacro:arg name="camera_model"  default="OAK-D-POE" />
-    <xacro:arg name="base_frame"    default="oak_base" />
-    <xacro:arg name="parent_frame"  default="oak_parent" />
-    <xacro:arg name="cam_pos_x"     default="0.0" />
-    <xacro:arg name="cam_pos_y"     default="0.0" />
-    <xacro:arg name="cam_pos_z"     default="0.0" />
-    <xacro:arg name="cam_roll"      default="0.0" />
-    <xacro:arg name="cam_pitch"     default="0.0" />
-    <xacro:arg name="cam_yaw"       default="0.0" />
-    <xacro:arg name="rs_compat"     default="true" />
-    <xacro:include filename="$(find depthai_descriptions)/urdf/depthai_descr.urdf.xacro" />
     <joint name="camera_base_joint" type="fixed">
         <parent link="base_link"/>
-        <child link="oak_parent"/>
+        <child link="zed_camera_link"/>
         <origin xyz="-0.05 -0.05 0.95" rpy="0 0 ${pi/2}"/>
     </joint>

Commit message: add zed camera link to description

File: src/igvc_description/urdf/sensor/camera.urdf.xacro (robot description, xacro)
@@ -1,4 +1,5 @@
 <?xml version="1.0" ?>
 <robot xmlns:xacro="http://www.ros.org/wiki/xacro">
+    <link name="zed_camera_link"/>
     <joint name="camera_base_joint" type="fixed">
         <parent link="base_link"/>

Commit message: Add zed to URDF

File: src/igvc_description/urdf/sensor/camera.urdf.xacro (robot description, xacro)
@@ -1,9 +1,10 @@
 <?xml version="1.0" ?>
 <robot xmlns:xacro="http://www.ros.org/wiki/xacro">
-    <link name="zed_camera_link"/>
-    <joint name="camera_base_joint" type="fixed">
-        <parent link="base_link"/>
-        <child link="zed_camera_link"/>
-        <origin xyz="-0.05 -0.05 0.95" rpy="0 0 ${pi/2}"/>
+    <xacro:include filename="$(find zed_wrapper)/urdf/zed_macro.urdf.xacro" />
+    <xacro:zed_camera name="zed" model="zed2i" />
+    <joint name="zed_camera_joint" type="fixed">
+        <parent link="base_link" />
+        <child link="zed_camera_link" />
+        <origin xyz="-0.05 -0.05 0.95" rpy="0 0 ${pi/2}" />
     </joint>
     <gazebo reference="oak_color_frame">

Commit message: change sensor angles

File: src/igvc_description/urdf/sensor/camera.urdf.xacro (robot description, xacro)
@@ -8,5 +8,5 @@
         <parent link="base_link" />
         <child link="zed_camera_link" />
-        <origin xyz="-0.05 -0.05 0.95" rpy="0 0 ${pi/2}" />
+        <origin xyz="-0.05 -0.05 0.95" rpy="0 ${12.5/180*pi} ${pi/2}" />
     </joint>
     <gazebo reference="oak_color_frame">

File: src/igvc_description/urdf/sensor/lidar.urdf.xacro (robot description, xacro)
@@ -4,5 +4,5 @@
         <parent link="base_link"/>
         <child link="laser_frame"/>
-        <origin xyz="-0.05 0.605 0.50" rpy="0 0 0"/>
+        <origin xyz="-0.05 0.605 0.50" rpy="0 0 ${-pi/2}"/>
     </joint>
     <link name="laser_frame">

Commit message: change zed positioning

File: src/igvc_description/urdf/sensor/camera.urdf.xacro (robot description, xacro)
@@ -6,7 +6,7 @@
     </xacro:zed_camera>
     <joint name="zed_camera_joint" type="fixed">
-        <parent link="base_link" />
+        <parent link="base_footprint" />
         <child link="zed_camera_link" />
-        <origin xyz="-0.05 -0.05 0.95" rpy="0 ${12.5/180*pi} ${pi/2}" />
+        <origin xyz="-0.05 -0.05 1.0033" rpy="0 ${11.5/180*pi} ${pi/2}" />
     </joint>
     <gazebo reference="oak_color_frame">

Commit message: remove placeholder camera positions

File: src/igvc_description/urdf/sensor/camera.urdf.xacro (robot description, xacro)
@@ -8,5 +8,5 @@
         <parent link="base_footprint" />
         <child link="zed_camera_link" />
-        <origin xyz="-0.05 -0.05 1.0033" rpy="0 ${11.5/180*pi} ${pi/2}" />
+        <origin xyz="0 0 1.0033" rpy="0 ${11.5/180*pi} ${pi/2}" />
     </joint>
     <gazebo reference="oak_color_frame">
